File: hardware/v2/ups12v/ups12v.kicad_pcb (KiCad board)
At the start: 4 copper layers, 21.6 x 21.6 mm, 5 parts, among them IC1 BQ25798RQMR, J2 BATTERY (BMS), Q1 SI2312CDS-T1-GE3, Q2 SI2312CDS-T1-GE3, Q3 SI2312CDS-T1-GE3

Commit message: temporary changes to PCB and schematics
Parts:
- removed Q3: SI2312CDS-T1-GE3, easyeda2kicad:SOT-23_L2.9-W1.3-P1.90-LS2.4-BR
- added C1: 47n 25V, Capacitor_SMD:C_0402_1005Metric, F.Cu at (61.5, 19.2)
- added C10: 10u 25V, Capacitor_SMD:C_0805_2012Metric, F.Cu at (65.1, 25.8)
- added C11: 10u 25V, Capacitor_SMD:C_0805_2012Metric, F.Cu at (65.1, 28.8)
- added C12: 10u 25V, Capacitor_SMD:C_0805_2012Metric, F.Cu at (65.1, 31.8)
- added C13: 10u 25V, Capacitor_SMD:C_0805_2012Metric, F.Cu at (69.6, 19.7)
- added C14: 10u 25V, Capacitor_SMD:C_0805_2012Metric, F.Cu at (69.6, 22.8)
- added C15: 10u 25V, Capacitor_SMD:C_0805_2012Metric, F.Cu at (69.6, 25.8)
- added C16: 10u 25V, Capacitor_SMD:C_0805_2012Metric, F.Cu at (69.6, 28.8)
- added C17: 10u 25V, Capacitor_SMD:C_0805_2012Metric, F.Cu at (69.6, 31.8)
- added C18: 10u 25V, Capacitor_SMD:C_0805_2012Metric, F.Cu at (74.0, 19.7)
- added C19: 10u 25V, Capacitor_SMD:C_0805_2012Metric, F.Cu at (74.0, 22.8)
- added C2: 47n 25V, Capacitor_SMD:C_0402_1005Metric, F.Cu at (61.5, 21.2)
- added C20: 47u POSCAP, easyeda2kicad:CASE-D_7343, F.Cu at (69.7, 37.5)
- added C21: 10u 25V, Capacitor_SMD:C_0805_2012Metric, F.Cu at (74.0, 25.8)
- added C22: 47u POSCAP, easyeda2kicad:CASE-D_7343, F.Cu at (69.7, 43.5)
- added C23: 47n 25V, Capacitor_SMD:C_0402_1005Metric, F.Cu at (61.5, 33.0)
- added C24: 47u low ESR, Capacitor_SMD:C_Elec_6.3x5.8, F.Cu at (55.0, 22.3)
- added C25: 47u low ESR, Capacitor_SMD:C_Elec_6.3x5.8, F.Cu at (55.0, 30.5)
- added C3: 4.7u 10V, Capacitor_SMD:C_0805_2012Metric, F.Cu at (65.1, 19.7)
- added C4: 10u 25V, Capacitor_SMD:C_0805_2012Metric, F.Cu at (65.1, 22.8)
- added C5: 100n 25V, Capacitor_SMD:C_0402_1005Metric, F.Cu at (61.5, 23.2)
- added C6: 100n 25V, Capacitor_SMD:C_0402_1005Metric, F.Cu at (61.5, 25.1)
- added C7: 100n 25V, Capacitor_SMD:C_0402_1005Metric, F.Cu at (61.5, 27.1)
- added C8: 1nF, 50V, Capacitor_SMD:C_0402_1005Metric, F.Cu at (61.5, 29.1)
- added C9: 100n 25V, Capacitor_SMD:C_0402_1005Metric, F.Cu at (61.5, 31.0)
- added D1: 12V, Diode_SMD:D_SOD-123, F.Cu at (64.9, 58.3)
- added D2: LED, LED_SMD:LED_0805_2012Metric, F.Cu at (70.1, 58.1)
- added H1: MountingHole, MountingHole:MountingHole_3.2mm_M3, F.Cu at (33.9, 22.2)
- added H2: MountingHole, MountingHole:MountingHole_3.2mm_M3, F.Cu at (33.9, 30.2)
- added H3: MountingHole, MountingHole:MountingHole_3.2mm_M3, F.Cu at (33.9, 38.1)
- added H4: MountingHole, MountingHole:MountingHole_3.2mm_M3, F.Cu at (33.9, 46.1)
- added J1: Input 12V DC, TerminalBlock_Phoenix:TerminalBlock_Phoenix_MKDS-1,5-2-5.08_1x02_P5.08mm_Horizontal, F.Cu at (41.4, 24.5)
- added J3: Battery, TerminalBlock_Phoenix:TerminalBlock_Phoenix_MKDS-1,5-2-5.08_1x02_P5.08mm_Horizontal, F.Cu at (41.4, 36.3)
- added J4: Conn_01x06_Pin, Connector_JST:JST_XH_B6B-XH-A_1x06_P2.50mm_Vertical, F.Cu at (63.0, 52.2)
- added J6: NTC temp sensor, Connector_JST:JST_XH_B2B-XH-A_1x02_P2.50mm_Vertical, F.Cu at (53.5, 52.2)
- added L1: 2.2uH, Inductor_SMD:L_12x12mm_H6mm, F.Cu at (57.5, 41.7)
- added NT1: ~, NetTie:NetTie-2_SMD_Pad0.5mm, F.Cu at (60.8, 57.3)
- added NT2: ~, NetTie:NetTie-2_SMD_Pad0.5mm, F.Cu at (60.8, 58.8)
- added NT4: ~, NetTie:NetTie-2_SMD_Pad0.5mm, F.Cu at (60.8, 60.3)
- added R1: 270R, Resistor_SMD:R_0805_2012Metric, F.Cu at (40.1, 43.4)
- added R4: 100R, Resistor_SMD:R_0805_2012Metric, F.Cu at (40.1, 46.4)
- added R5: 27k 1-2%, Resistor_SMD:R_0805_2012Metric, F.Cu at (40.1, 49.3)
- added R6: 5k6, Resistor_SMD:R_0805_2012Metric, F.Cu at (40.1, 52.3)
- added R7: 33k, Resistor_SMD:R_0805_2012Metric, F.Cu at (40.1, 55.2)
- added R8: 2k2, Resistor_SMD:R_0805_2012Metric, F.Cu at (40.1, 58.2)
- added R9: 10k, Resistor_SMD:R_0805_2012Metric, F.Cu at (40.1, 61.1)
- added TP1: GND, TestPoint:TestPoint_Loop_D1.80mm_Drill1.0mm_Beaded, F.Cu at (44.6, 44.3)
- added TP3: PGND, TestPoint:TestPoint_Loop_D1.80mm_Drill1.0mm_Beaded, F.Cu at (44.6, 48.9)
- added TP4: SYS, TestPoint:TestPoint_Loop_D1.80mm_Drill1.0mm_Beaded, F.Cu at (44.6, 53.6)
- added TP8: REGN, TestPoint:TestPoint_Loop_D1.80mm_Drill1.0mm_Beaded, F.Cu at (44.6, 58.2)
- added U1: mini_esp32 MH-ET-Live, Modules_MCU:ESP32_mini MH-ET-LIVE, F.Cu at (96.8, 37.8)
- IC1: footprint mouser (samacsys):BQ25798RQMR -> mouser (samacsys):BQ25798RQMR_smaller_protected_area
- J2: value BATTERY (BMS) -> Output 12V DC
- Q1, Q2: value SI2312CDS-T1-GE3 -> AON7528; footprint easyeda2kicad:SOT-23_L2.9-W1.3-P1.90-LS2.4-BR -> easyeda2kicad:DFN-8_L3.3-W3.3-P0.65-BL-3
Connections:
- net BAT renamed BATTERY
- IC1 pad 11: Net-(IC1-ACDRV1) -> (no net)
- IC1 pad 12: unconnected-(IC1-~{QON}-Pad12) -> (no net)
- IC1 pad 13: GND -> /BQ25798 module/~RST
- IC1 pad 14: I2C_SCL -> /BQ25798 module/I2C_SCL
- IC1 pad 15: I2C_SDA -> /BQ25798 module/I2C_SDA
- IC1 pad 18: BATP -> (no net)
- IC1 pad 2: VBUS -> (no net)
- IC1 pad 20: Net-(IC1-PROG) -> (no net)
- IC1 pad 21: unconnected-(IC1-~{INT}-Pad21) -> /BQ25798 module/~INT
- IC1 pad 25: Net-(IC1-SYS) -> SYS
- IC1 pad 27: GND -> PGND
- IC1 pad 29: Net-(IC1-PMID) -> PMID
- IC1 pad 3: VBUS -> (no net)
- IC1 pad 6: unconnected-(IC1-D+-Pad6) -> (no net)
- IC1 pad 7: unconnected-(IC1-D--Pad7) -> (no net)
- IC1 pad 8: VBUS -> (no net)
- J2 pad 1: Net-(J2-Pin_1) -> PGND
- J2 pad 2: GND -> PMID
- Q1 pad 1: Net-(D1-K) -> (no net)
- Q1 pad 2: Net-(D1-A) -> (no net)
- Q1 pad 3: VIN1 -> (no net)
- Q2 pad 1: Net-(D1-K) -> (no net)
- Q2 pad 2: Net-(D1-A) -> (no net)
- Q2 pad 3: VBUS -> (no net)
