File: hardware/v2/bq25798_module/bq25798_module.kicad_sch (KiCad schematic)
At the start: 54 parts, among them IC1 BQ25798RQMR, J1 Input 12V DC, J2 Output 12V DC, J3 Battery, J4 Conn_01x06_Pin, J6 NTC temp sensor, Q1 AON7528, Q2 AON7528

Commit message: wip ESP32 schematics
Parts:
- added C26: 470u 50V, Capacitor_SMD:C_0805_2012Metric, symbol Device:C
- added C27: 220u 25V, Capacitor_SMD:C_0805_2012Metric, symbol Device:C
- added C28: 10u 25V, Capacitor_SMD:C_0805_2012Metric, symbol Device:C
- added J5: USB_C_Receptacle_USB2.0_14P, Connector_USB:USB_C_Receptacle_HCTL_HC-TYPE-C-16P-01A, symbol Connector:USB_C_Receptacle_USB2.0_14P
- added L2: 68 uH, mouser (samacsys):INDPM7676X435N, symbol Device:L_Small
- added R2, R3: 5k1, Resistor_SMD:R_0805_2012Metric, symbol Device:R
- added U1: ESP32-S2-WROVER, RF_Module:ESP32-S2-WROVER, symbol RF_Module:ESP32-S2-WROVER
- added U2: LM2596S-3.3, Package_TO_SOT_SMD:TO-263-5_TabPin3, symbol Regulator_Switching:LM2596S-3.3
Connections:
- net GND: now also C26.2, C27.2, C28.2, J5.A1 (GND), J5.A12 (GND), J5.B1 (GND), J5.B12 (GND), J5.S1 (SHIELD), R2.1, R3.1, U1.1 (GND), U1.26 (GND), U1.42 (GND), U1.43 (GND), U2.3 (GND), U2.5 (~{ON}/OFF)
- new net: C26.1, J5.A4 (VBUS), J5.A9 (VBUS), J5.B4 (VBUS), J5.B9 (VBUS), U2.1 (VIN)
- new net: L2.2, U2.2 (OUT)
- new net: C27.1, C28.1, L2.1, U1.2 (3V3), U2.4 (FB)
- new net: J5.A7 (D-), J5.B7 (D-), U1.22 (USB_D-)
- new net: J5.A6 (D+), J5.B6 (D+), U1.23 (USB_D+)
- new net: J5.A5 (CC1), R2.2
- new net: J5.B5 (CC2), R3.2
- no-connect marks 3 -> 39
