File: hardware/v2/bq25798_module/bq25798_module.kicad_pcb (KiCad board)
At the start: 4 copper layers, 76 x 55.9 mm, 65 parts, among them IC1 BQ25798RQMR, J1 Input 12V DC, J2 Output 12V DC, J3 Battery, J4 Conn_01x06_Pin, J6 NTC temp sensor, Q1 AON7528, Q2 AON7528

Commit message: v3.3b
Parts:
- removed TP8: REGN, TestPoint:TestPoint_Loop_D1.80mm_Drill1.0mm_Beaded
- removed kibuzzard-683C9D12: G***, kibuzzard-683C9D12
- added kibuzzard-68585403: G***, kibuzzard-68585403, F.Cu at (106.4, 89.9)
Routing:
- net REGN: track 58.8 -> 52.2 mm
Other:
- outline, holes or cut-outs redrawn
- board text added: "1S = 4k7 2S = 8k2 3S = 13k7 4S = 27k"
- board text added: "BQ25798 UPS V3.3b by Michal Schwarz"
- board text removed: "BQ25798 UPS V3.3 by Michal Schwarz"
