File: hardware/v2/controller/controller.kicad_pcb (KiCad board)
At the start: 2 copper layers, 76 x 55.9 mm, 15 parts, among them J1 I2C etc., U1 mini_esp32 MH-ET-Live, U2 Micro step down converter

Commit message: update controller board too
Parts:
- moved kibuzzard-6810F062 42.3 mm to (155.2, 77.0), turned to -90 degrees
- moved kibuzzard-6810F0D5 38.7 mm to (157.8, 76.7), turned to -90 degrees
- moved kibuzzard-6810F0CD 35.1 mm to (160.3, 76.7), turned to -90 degrees
- moved kibuzzard-6810EFE9 31.7 mm to (162.7, 77.0), turned to -90 degrees
- moved kibuzzard-6810F0BF 28.1 mm to (165.3, 77.0), turned to -90 degrees
- moved kibuzzard-683D9CD5 24.7 mm to (167.7, 76.7), turned to -90 degrees
- moved U1 17.7 mm to (132.1, 101.6), turned to 90 degrees
- moved J1 15.7 mm to (167.6, 83.2), turned to 180 degrees
- moved R2 9.92 mm to (160.0, 90.4), turned to 90 degrees
- moved R1 6.83 mm to (163.1, 90.4), turned to 90 degrees
- moved U2 0.58 mm to (176.2, 126.2)
Routing:
- net /I2C_SCL: track 74.7 -> 44.1 mm, vias 1 -> 0
- net /I2C_SDA: track 61.2 -> 44.4 mm, vias 1 -> 2
- net /~INT: track 46.7 -> 34.7 mm, vias 0 -> 1
- net /PWR_IN: track 34.2 -> 45.4 mm
- net /~RST: track 47.8 -> 36.7 mm
- net 3V3: track 67.8 -> 68.4 mm
- net GND: vias 0 -> 6
Other:
- outline, holes or cut-outs redrawn
- board text added: "BQ25798 UPS Controller V1.1 by Michal Schwarz"
- board text removed: "BQ25798 UPS Controller V1.0 by Michal Schwarz"
