File: hardware/v4/ups_v4/ups12v_v4.kicad_sch (KiCad schematic)
At the start: 59 parts, among them IC1 BQ25798RQMR, J1 ADAPTER 4.75-21V, J2 VSYS OUTPUT, J3 BATTERY 2S/4S, J4 MCU / BIAS INTERFACE, J6 NTC temp sensor, Q1 AON7528, Q2 AON7528, Q3 PMV16UN

Commit message: next stage
Parts:
- C10, C11, C14, C17, C19, C21, C4: MPN (none) -> GRJ21BR61E106KE01K; Manufacturer (none) -> Murata; MetadataEvidence (none) -> V4_STAGE2_PARTS.md; Murata GRJ21BR61E106KE01-02A, 2024-12-10; Parameters X7R -> X5R; +/-10%; -55 to +85 degC; VoltageRating (none) -> 25V
- C8: MPN (none) -> GCM1555C1H102JA16D; Manufacturer (none) -> Murata; MetadataEvidence (none) -> V4_STAGE2_PARTS.md; Murata GCM1555C1H102JA16-01A, 2022-04-08; Parameters X7R -> C0G (NP0); +/-5%; -55 to +125 degC; VoltageRating (none) -> 50V
- R5: value 27k 1-2% -> 27k 1%; AssemblyProfiles (none) -> 27k: S792-4/S798-4; 8.2k: S792-2/S798-2; both 1%, 750kHz; SelectionStatus (none) -> Fixed assembly population; exact MPN OPEN; no cell-count ju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

Commit message: phase 2.6
Parts:
- added C26: 2.2u 100V X7R, Capacitor_SMD:C_1210_3225Metric, symbol Device:C
- added R12: 2R 5% pulse, Resistor_SMD:R_1206_3216Metric, symbol Device:R
- F1: ApprovalStatus (none) -> PROPOSED; FootprintEvidence (none) -> phase2-6-fuse-readback.json; manufacturer GD.12/01/25 p4, i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
Connections:
- net PGND: now also C26.2
- net VIN1: now also R12.1
- new net: C26.1, R12.2
Other:
- note added: "VIN hot-plug RC: TI Fig. 8-1 (>15V) Provisional R12 / C26; validate on prototype"
- moved on the sheet: IC1, J2

Commit message: phase 3.1
Parts:
- added C27: 10u 6.3V USB VBUS, Capacitor_SMD:C_0805_2012Metric, symbol Device:C
- added C28: 100n 10V USB VBUS, Capacitor_SMD:C_0402_1005Metric, symbol Device:C
- added C29: 1u RESET RC (PROVISIONAL), Capacitor_SMD:C_0402_1005Metric, symbol Device:C
- added C30: 10u MCU3V3 BULK (PROVISIONAL), Capacitor_SMD:C_0805_2012Metric, symbol Device:C
- added C31: 100n MCU3V3 HF (PROVISIONAL), Capacitor_SMD:C_0402_1005Metric, symbol Device:C
- added J7: USB-C PROGRAM / NATIVE USB, Connector_USB:USB_C_Receptacle_GCT_USB4105-xx-A_16P_TopMnt_Horizontal, symbol Connector:USB_C_Receptacle_USB2.0_16P
- added R13, R14: 5k1 1%, Resistor_SMD:R_0402_1005Metric, symbol Device:R
- added R15: 10k 1% BOOT, Resistor_SMD:R_0402_1005Metric, symbol Device:R
- added R16: 10k 1% EN, Resistor_SMD:R_0402_1005Metric, symbol Device:R
- added R17: 10k 1% GPIO2, Resistor_SMD:R_0402_1005Metric, symbol Device:R
- added R18: 10k 1% GPIO8, Resistor_SMD:R_0402_1005Metric, symbol Device:R
- added SW1: BOOT / DOWNLOAD, Button_Switch_SMD:SW_SPST_EVQP0, symbol Switch:SW_Push
- added SW2: RESET, Button_Switch_SMD:SW_SPST_EVQP0, symbol Switch:SW_Push
- added U1: ESP32-C3-MINI-1-N4X (PROVISIONAL), Modules_MCU:ESP32-C3-MINI-1, symbol ups_v4_custom:ESP32-C3-MINI-1
- added U2: TPD2EUSB30A (PROVISIONAL), Package_TO_SOT_SMD:SOT-23, symbol Power_Protection:TPD2EUSB30A
Connections:
- net PGND: now also C27.2, C28.2, C29.2, C30.2, C31.2, J7.A1 (GND), J7.A12 (GND), J7.B1 (GND), J7.B12 (GND), J7.SH (SHIELD), R13.2, R14.2, SW1.2, SW2.2, U1.1 (GND), U1.11 (GND), U1.14 (GND), U1.2 (GND), U1.36 (GND), U1.37 (GND), U1.38 (GND), U1.39 (GND), U1.40 (GND), U1.41 (GND), U1.42 (GND), U1.43 (GND), U1.44 (GND), U1.45 (GND), U1.46 (GND), U1.47 (GND), U1.48 (GND), U1.49 (GND), U1.50 (GND), U1.51 (GND), U1.52 (GND), U1.53 (GND), U2.3 (GND)
- new net MCU3V3: C30.1, C31.1, R15.2, R16.2, R17.2, R18.2, U1.3 (3V3)
- new net MCU_BOOT: R15.1, SW1.1, U1.23 (GPIO9)
- new net MCU_BOOT_STRAP2: R17.1, U1.5 (GPIO2)
- new net MCU_BOOT_STRAP8: R18.1, U1.22 (GPIO8)
- new net MCU_CHG_ARM: U1.21 (GPIO7)
- new net MCU_EN: C29.1, R16.1, SW2.1, U1.8 (EN)
- new net MCU_GPIO0: U1.12 (GPIO0)
- new net MCU_GPIO1: U1.13 (GPIO1)
- new net MCU_GPIO10: U1.16 (GPIO10)
- new net MCU_INT: U1.20 (GPIO6)
- new net MCU_SCL: U1.19 (GPIO5)
- new net MCU_SDA: U1.18 (GPIO4)
- new net MCU_STATUS_LED: U1.6 (GPIO3)
- new net UART_RX: U1.30 (UART_RX / GPIO20)
- new net UART_TX: U1.31 (UART_TX / GPIO21)
- new net USB_CC1: J7.A5 (CC1), R13.1
- new net USB_CC2: J7.B5 (CC2), R14.1
- new net USB_DN: J7.A7 (D-), J7.B7 (D-), U1.26 (USB_D- / GPIO18), U2.2 (D-)
- new net USB_DP: J7.A6 (D+), J7.B6 (D+), U1.27 (USB_D+ / GPIO19), U2.1 (D+)
- new net USB_VBUS: C27.1, C28.1, J7.A4 (VBUS), J7.A9 (VBUS), J7.B4 (VBUS), J7.B9 (VBUS)
- no-connect marks 3 -> 19
Other:
- note added: "MCU3V3 is a reserved power-domain input; VSYS buck, USB buck and mux are pending next checkpoint."
- note added: "PCB BLOCK: exact Espressif land-pattern comparison pending; readback is 62 physical pads / 60 unique numbers, duplicate ground numbers, no courtyard."
- note added: "PHASE 3.1 CHECKPOINT: native USB / recovery wiring only"
- note added: "USB_VBUS is USB-only input; USB-derived 3V3 regulator is pending next checkpoint."

Commit message: phase 3-2
Parts:
- added C32: 2.2u NORMAL IN, Capacitor_SMD:C_0805_2012Metric, symbol Device:C
- added C33: 22u NORMAL OUT, Capacitor_SMD:C_0805_2012Metric, symbol Device:C
- added C34: 2.2u USB IN, Capacitor_SMD:C_0805_2012Metric, symbol Device:C
- added C35: 22u USB OUT, Capacitor_SMD:C_0805_2012Metric, symbol Device:C
- added C36: 22u MCU3V3 BULK, Capacitor_SMD:C_0805_2012Metric, symbol Device:C
- added C37: 100n NORMAL BOOST, Capacitor_SMD:C_0402_1005Metric, symbol Device:C
- added C38: 100n USB BOOST, Capacitor_SMD:C_0402_1005Metric, symbol Device:C
- added C39: 33n NORMAL SS, Capacitor_SMD:C_0402_1005Metric, symbol Device:C
- added C40: 33n USB SS, Capacitor_SMD:C_0402_1005Metric, symbol Device:C
- added C41: 100n MCU UV, Capacitor_SMD:C_0402_1005Metric, symbol Device:C
- added C42: 10n SUP CT, Capacitor_SMD:C_0402_1005Metric, symbol Device:C
- added C43: 100n NORMAL VIN, Capacitor_SMD:C_0402_1005Metric, symbol Device:C
- added C44: 100n USB VIN, Capacitor_SMD:C_0402_1005Metric, symbol Device:C
- added C45: 22u NORMAL OUT 2, Capacitor_SMD:C_0805_2012Metric, symbol Device:C
- added C46: 22u USB OUT 2, Capacitor_SMD:C_0805_2012Metric, symbol Device:C
- added C47: 100n MCU TCA VCCB, Capacitor_SMD:C_0402_1005Metric, symbol Device:C
- added C48: 100n MAIN TCA VCCA, Capacitor_SMD:C_0402_1005Metric, symbol Device:C
- added C49: 470u MCU HOLDUP, Capacitor_SMD:C_Elec_8x10.2, symbol Device:C_Polarized
- added C50: 47n 30V TPS22975 CT, Capacitor_SMD:C_0402_1005Metric, symbol Device:C
- added C51: 22u PRE-MUX 6.3V, Capacitor_SMD:C_0805_2012Metric, symbol Device:C
- added C52: 10n MCU UV CT, Capacitor_SMD:C_0402_1005Metric, symbol Device:C
- added D5: BAT54W RESET ISOLATION, Diode_SMD:D_SOD-323, symbol Device:D
- added L2: 4.7uH XAL5030 NORMAL, Inductor_SMD:L_Coilcraft_XAL5030-XXX, symbol Device:L
- added L3: 4.7uH XAL5030 USB, Inductor_SMD:L_Coilcraft_XAL5030-XXX, symbol Device:L
- added Q10: BC847 MCU ARM LIVE SINK, Package_TO_SOT_SMD:SOT-23, symbol Transistor_BJT:BC847
- added Q4: BC847 INT DOMAIN ISOLATOR, Package_TO_SOT_SMD:SOT-23, symbol Transistor_BJT:BC847
- added Q5: BC857 MAIN-GATED CHG SOURCE, Package_TO_SOT_SMD:SOT-23, symbol Transistor_BJT:BC857
- added Q6: BC847 MAIN_VALID SINK, Package_TO_SOT_SMD:SOT-23, symbol Transistor_BJT:BC847
- added Q7: BC847 MCU CHG ARM SINK, Package_TO_SOT_SMD:SOT-23, symbol Transistor_BJT:BC847
- added Q8: PMV16UN MAIN_VALID, Package_TO_SOT_SMD:SOT-23, symbol Transistor_FET:2N7002
- added Q9: PMV16UN TCA_EN, Package_TO_SOT_SMD:SOT-23, symbol Transistor_FET:2N7002
- added R19: 4k7 MCU I2C SCL PU, Resistor_SMD:R_0402_1005Metric, symbol Device:R
- added R20: 4k7 MCU I2C SDA PU, Resistor_SMD:R_0402_1005Metric, symbol Device:R
- added R21: 4k7 MAIN I2C SCL PU, Resistor_SMD:R_0402_1005Metric, symbol Device:R
- added R22: 4k7 MAIN I2C SDA PU, Resistor_SMD:R_0402_1005Metric, symbol Device:R
- added R23: 10k MAIN_VALID PULLUP, Resistor_SMD:R_0402_1005Metric, symbol Device:R
- added R25: 100k MUX ST PU, Resistor_SMD:R_0402_1005Metric, symbol Device:R
- added R28: 10k MAIN INT PU, Resistor_SMD:R_0402_1005Metric, symbol Device:R
- added R29: 10k INT BASE, Resistor_SMD:R_0402_1005Metric, symbol Device:R
- added R30: 100k INT BASE PD, Resistor_SMD:R_0402_1005Metric, symbol Device:R
- added R31: 4k7 MCU INT PU, Resistor_SMD:R_0402_1005Metric, symbol Device:R
- added R32: 32k2 0.1% NORMAL FB, Resistor_SMD:R_0402_1005Metric, symbol Device:R
- added R33: 10k 0.1% NORMAL FB, Resistor_SMD:R_0402_1005Metric, symbol Device:R
- added R34: 32k2 0.1% USB FB, Resistor_SMD:R_0402_1005Metric, symbol Device:R
- added R35: 10k 0.1% USB FB, Resistor_SMD:R_0402_1005Metric, symbol Device:R
- added R36: 100k NORMAL EN, Resistor_SMD:R_0402_1005Metric, symbol Device:R
- added R37: 38k3 NORMAL EN, Resistor_SMD:R_0402_1005Metric, symbol Device:R
- added R38: 100k USB EN, Resistor_SMD:R_0402_1005Metric, symbol Device:R
- added R39: 47k USB EN, Resistor_SMD:R_0402_1005Metric, symbol Device:R
- added R44: 100k CHG BASE PU, Resistor_SMD:R_0402_1005Metric, symbol Device:R
- added R46: 4k7 MCU CHG BASE, Resistor_SMD:R_0402_1005Metric, symbol Device:R
- added R47: 100k MCU CHG BASE PD, Resistor_SMD:R_0402_1005Metric, symbol Device:R
- added R48: 0R USB_DP SERIES (22R OPTION), Resistor_SMD:R_0402_1005Metric, symbol Device:R
- added R49: 0R USB_DN SERIES (22R OPTION), Resistor_SMD:R_0402_1005Metric, symbol Device:R
- added R50: 100k MAIN_VALID TO Q6 BASE, Resistor_SMD:R_0402_1005Metric, symbol Device:R
- added R51: 100k NEN PU, Resistor_SMD:R_0402_1005Metric, symbol Device:R
- added R52: 100k TCA_EN PU, Resistor_SMD:R_0402_1005Metric, symbol Device:R
- added R53: 10k Q5 BASE LIMIT, Resistor_SMD:R_0402_1005Metric, symbol Device:R
- added R54: 100k CHG LATCH CLR PU, Resistor_SMD:R_0402_1005Metric, symbol Device:R
- added R55: 100k MCU ARM PD, Resistor_SMD:R_0402_1005Metric, symbol Device:R
- added R56: 16k7 0.1% MCU UV TOP, Resistor_SMD:R_0402_1005Metric, symbol Device:R
- added R57: 10k 0.1% MCU UV BOT, Resistor_SMD:R_0402_1005Metric, symbol Device:R
- added U10: TPS22975DSGR MCU3V3 SOFTSTART, Package_SON:Texas_DSG0008A_WSON-8-1EP_2x2mm_P0.5mm_EP0.9x1.6mm, symbol ups_v4_custom:TPS22975
- added U11: TPS389001DSET MCU UV, Package_SON:WSON-6_1.5x1.5mm_P0.5mm, symbol ups_v4_custom:TPS389033C
- added U12: SN74LVC1G17DBVR CLR SCHMITT, Package_TO_SOT_SMD:SOT-23-5, symbol 74xGxx:74LVC1G17
- added U3: TPS62933DRLR NORMAL 3V3, Package_TO_SOT_SMD:SOT-583-8, symbol Regulator_Switching:TPS62933
- added U4: TPS62933DRLR USB 3V3, Package_TO_SOT_SMD:SOT-583-8, symbol Regulator_Switching:TPS62933
- added U5: TPS2116DRL NORMAL PRIORITY, Package_TO_SOT_SMD:SOT-583-8, symbol Power_Management:TPS2116DRL
- added U6: TCA9517DGKR REV.D, Package_SO:VSSOP-8_3x3mm_P0.65mm, symbol Logic_LevelTranslator:TCA9517ADGK
- added U7: TPS389033DSET MAIN UV, Package_SON:WSON-6_1.5x1.5mm_P0.5mm, symbol ups_v4_custom:TPS389033C
- added U8: TPS389033DSET USB ARM UV, Package_SON:WSON-6_1.5x1.5mm_P0.5mm, symbol ups_v4_custom:TPS389033C
- added U9: SN74LVC1G74DCTR CHG LATCH, Package_SO:SSOP-8_2.95x2.8mm_P0.65mm, symbol ups_v4_custom:SN74LVC1G74
- R11: value 1k -> 4k7 SERVICE CHG_REQ SENSE DNP; DNP (none) -> YES; Parameters (none) -> External CHG_REQ retained at J4 for service observation onl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; PopulationGroup (none) -> Service-only CHG_REQ sense; DNP; does not enable charge
- U1: value ESP32-C3-MINI-1-N4X (PROVISIONAL) -> ESP32-C3-MINI-1-N4X; footprint Modules_MCU:ESP32-C3-MINI-1 -> ups_v4:ESP32-C3-MINI-1-N4X; FootprintReview BLOCKED: footprint readback has 62 physical pads / 60 uniqu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 -> PASS READBACK: project-local N4X footprint has 61 physical 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; Parameters (none) -> GPIO0/pad12 is MCU_CHG_ARM; GPIO7/pad21 is MCU_GPIO7; firmw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
- U2: footprint Package_TO_SOT_SMD:SOT-23 -> Package_TO_SOT_SMD:Texas_DRT-3
Connections:
- net MCU_GPIO0 is gone; now on net MCU_CHG_ARM: U1.12 (GPIO0)
- net CHG_GATE: now also Q5.3 (C); no longer R11.2
- net I2C_SCL: now also R21.2, U6.2 (SCLA)
- net I2C_SDA: now also R22.2, U6.3 (SDAA)
- net MAIN_3V3: now also C33.1, C45.1, C48.1, L2.2, Q5.2 (E), R21.1, R22.1, R23.1, R28.1, R32.1, R44.1, U5.3 (VIN1), U5.5 (MODE), U6.1 (VCCA), U7.1 (SENSE), U7.3 (MR), U7.4 (VDD), U8.1 (SENSE)
- net MCU3V3: now also C36.1, C41.1, C47.1, C49.1, R19.1, R20.1, R25.1, R31.1, R51.1, R52.1, R54.1, R56.1, U10.7 (VOUT), U10.8 (VOUT), U11.3 (MR), U11.4 (VDD), U12.5 (VCC), U6.8 (VCCB), U8.3 (MR), U8.4 (VDD), U9.2 (D), U9.7 (PRE), U9.8 (VCC)
- net MCU_CHG_ARM: now also R46.1, U9.1 (CLK); no longer U1.21 (GPIO7)
- net MCU_EN: now also D5.1 (K), U11.6 (RESET)
- net MCU_INT: now also Q4.3 (C), R31.2
- net MCU_SCL: now also R19.2, U6.7 (SCLB)
- net MCU_SDA: now also R20.2, U6.6 (SDAB)
- net PGND: now also C32.2, C33.2, C34.2, C35.2, C36.2, C39.2, C40.2, C41.2, C42.2, C43.2, C44.2, C45.2, C46.2, C47.2, C48.2, C49.2, C50.2, C51.2, C52.2, Q10.2 (E), Q4.2 (E), Q8.2 (S), Q9.2 (S), R30.2, R33.2, R35.2, R37.2, R39.2, R47.2, R55.2, R57.2, U10.5 (GND), U11.2 (GND), U12.3 (GND), U3.4 (GND), U4.4 (GND), U5.1 (GND), U6.4 (GND), U7.2 (GND), U8.2 (GND), U8.5 (CT), U9.4 (GND)
- net SYS: now also C32.1, C43.1, R36.1, U3.3 (VIN)
- net USB_DN: now also R49.2; no longer U1.26 (USB_D- / GPIO18)
- net USB_DP: now also R48.2; no longer U1.27 (USB_D+ / GPIO19)
- net USB_VBUS: now also C34.1, C44.1, R38.1, U4.3 (VIN)
- net ~INT: now also R28.2, R29.1
- new net: Q6.1 (B), R50.2
- new net: R49.1, U1.26 (USB_D- / GPIO18)
- new net: R48.1, U1.27 (USB_D+ / GPIO19)
- new net BST_NORMAL: C37.1, U3.6 (BST)
- new net BST_USB: C38.1, U4.6 (BST)
- new net CHG_AND: Q6.2 (E), Q7.3 (C)
- new net CHG_BASE: Q6.3 (C), R53.1
- new net CHG_LATCH: Q7.1 (B), R47.1, U9.5 (Q)
- new net CHG_LATCH_CLR_N: D5.2 (A), R54.2, U12.2, U8.6 (RESET)
- new net CHG_LATCH_CLR_SCHMITT_N: U12.4, U9.6 (CLR)
- new net CHG_LIVE_AND: Q10.3 (C), Q7.2 (E)
- new net INT_BASE: Q4.1 (B), R29.2, R30.1
- new net MAIN_FB: R32.2, R33.1, U3.8 (FB)
- new net MCU_CHG_LIVE: Q10.1 (B), R46.2, R55.1
- new net MCU_GPIO7: U1.21 (GPIO7)
- new net MCU_PRE3V3: C51.1, U10.1 (VIN), U10.2 (VIN), U10.3 (ON), U10.4 (VBIAS), U5.2 (VOUT), U5.7 (VOUT)
- new net MCU_UV_CT: C52.1, U11.5 (CT)
- new net MCU_UV_SENSE: R56.2, R57.1, U11.1 (SENSE)
- new net MUX_PR1: Q8.1 (G), R23.2, R50.1, U5.4 (PR1), U7.6 (RESET)
- new net MUX_ST: R25.2, U5.8 (ST)
- new net NEN: Q8.3 (D), Q9.1 (G), R51.2
- new net NORMAL_EN: R36.2, R37.1, U3.2 (EN)
- new net NORMAL_SS: C39.1, U3.7 (SS)
- new net Q5_BASE_LIMITED: Q5.1 (B), R44.2, R53.2
- new net SW_NORMAL: C37.2, L2.1, U3.5 (SW)
- new net SW_USB: C38.2, L3.1, U4.5 (SW)
- new net TCA_EN: Q9.3 (D), R52.2, U6.5 (EN)
- new net TPS22975_CT: C50.1, U10.6 (CT)
- new net TPS3890_CT: C42.1, U7.5 (CT)
- new net USB3V3: C35.1, C46.1, L3.2, R34.1, U5.6 (VIN2)
- new net USB_EN: R38.2, R39.1, U4.2 (EN)
- new net USB_FB: R34.2, R35.1, U4.8 (FB)
- new net USB_SS: C40.1, U4.7 (SS)
- no-connect marks 19 -> 24

Commit message: phase 3.3 and 3.4
Parts:
- removed C34: 2.2u USB IN, Capacitor_SMD:C_0805_2012Metric, symbol Device:C
- removed C38: 100n USB BOOST, Capacitor_SMD:C_0402_1005Metric, symbol Device:C
- removed C41: 100n MCU UV, Capacitor_SMD:C_0402_1005Metric, symbol Device:C
- removed C42: 10n SUP CT, Capacitor_SMD:C_0402_1005Metric, symbol Device:C
- removed C44: 100n USB VIN, Capacitor_SMD:C_0402_1005Metric, symbol Device:C
- removed C46: 22u USB OUT 2, Capacitor_SMD:C_0805_2012Metric, symbol Device:C
- removed C49: 470u MCU HOLDUP, Capacitor_SMD:C_Elec_8x10.2, symbol Device:C_Polarized
- removed C50: 47n 30V TPS22975 CT, Capacitor_SMD:C_0402_1005Metric, symbol Device:C
- removed C51: 22u PRE-MUX 6.3V, Capacitor_SMD:C_0805_2012Metric, symbol Device:C
- removed C52: 10n MCU UV CT, Capacitor_SMD:C_0402_1005Metric, symbol Device:C
- removed D5: BAT54W RESET ISOLATION, Diode_SMD:D_SOD-323, symbol Device:D
- removed L3: 4.7uH XAL5030 USB, Inductor_SMD:L_Coilcraft_XAL5030-XXX, symbol Device:L
- removed Q10: BC847 MCU ARM LIVE SINK, Package_TO_SOT_SMD:SOT-23, symbol Transistor_BJT:BC847
- removed R34: 32k2 0.1% USB FB, Resistor_SMD:R_0402_1005Metric, symbol Device:R
- removed R38: 100k USB EN, Resistor_SMD:R_0402_1005Metric, symbol Device:R
- removed R39: 47k USB EN, Resistor_SMD:R_0402_1005Metric, symbol Device:R
- removed R54: 100k CHG LATCH CLR PU, Resistor_SMD:R_0402_1005Metric, symbol Device:R
- removed R55: 100k MCU ARM PD, Resistor_SMD:R_0402_1005Metric, symbol Device:R
- removed R56: 16k7 0.1% MCU UV TOP, Resistor_SMD:R_0402_1005Metric, symbol Device:R
- removed R57: 10k 0.1% MCU UV BOT, Resistor_SMD:R_0402_1005Metric, symbol Device:R
- removed U10: TPS22975DSGR MCU3V3 SOFTSTART, Package_SON:Texas_DSG0008A_WSON-8-1EP_2x2mm_P0.5mm_EP0.9x1.6mm, symbol ups_v4_custom:TPS22975
- removed U11: TPS389001DSET MCU UV, Package_SON:WSON-6_1.5x1.5mm_P0.5mm, symbol ups_v4_custom:TPS389033C
- removed U12: SN74LVC1G17DBVR CLR SCHMITT, Package_TO_SOT_SMD:SOT-23-5, symbol 74xGxx:74LVC1G17
- removed U4: TPS62933DRLR USB 3V3, Package_TO_SOT_SMD:SOT-583-8, symbol Regulator_Switching:TPS62933
- removed U7: TPS389033DSET MAIN UV, Package_SON:WSON-6_1.5x1.5mm_P0.5mm, symbol ups_v4_custom:TPS389033C
- removed U8: TPS389033DSET USB ARM UV, Package_SON:WSON-6_1.5x1.5mm_P0.5mm, symbol ups_v4_custom:TPS389033C
- removed U9: SN74LVC1G74DCTR CHG LATCH, Package_SO:SSOP-8_2.95x2.8mm_P0.65mm, symbol ups_v4_custom:SN74LVC1G74
- added R24: 4k7 1% MAIN_VALID DIVIDER BOTTOM, Resistor_SMD:R_0402_1005Metric, symbol Device:R
- added U4: AP7361C-33E-13 USB 3V3 LDO, Package_TO_SOT_SMD:SOT-223-3_TabPin2, symbol Regulator_Linear:AP7361C-33E
- C27: value 10u 6.3V USB VBUS -> 4.7u 10V USB LDO IN
- C40: value 33n USB SS -> 100n USB LDO OUT
- R23: value 10k MAIN_VALID PULLUP -> 8k2 1% MAIN_VALID DIVIDER TOP; Parameters 10k 1% MAIN_3V3 pull-up for TPS389033 RESET/MUX_PR1; digita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 -> 8k2 1% MAIN-referenced TPS2116 PR1 divider top; priority th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
- R35: value 10k 0.1% USB FB -> 10k USB3V3 BLEED; ApprovalStatus (none) -> PROPOSED; Parameters (none) -> 10k USB3V3-to-PGND bleeder; approx 0.33mA at 3.3V; bounds u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; PopulationGroup (none) -> USB service regulator support
- R50: Parameters 100k candidate; supervisor-released MUX_PR1 drives Q6 base;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 -> 100k MAIN_3V3 to Q6 base; direct main-domain bias; exact lo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; PopulationGroup MAIN_VALID to Q6 base authorization resistor -> MAIN-domain isolation bias resistor
- U5: Parameters VIN1 normal priority; VIN2 USB; 1.6-5.5V; 2.5A; PR1=10k MAI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 -> VIN1 MAIN_3V3 normal priority; VIN2 USB3V3 service; MODE=MA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
Connections:
- net CHG_LIVE_AND is gone; now on net PGND: Q7.2 (E)
- net MCU_CHG_LIVE is gone; now on net MCU_CHG_BASE: R46.2
- net MCU_PRE3V3 is gone; now on net MCU3V3: U5.2 (VOUT), U5.7 (VOUT)
- net USB_FB is gone; now on net USB3V3: R35.1
- net USB_SS is gone; now on net USB3V3: C40.1
- net MAIN_3V3: now also Q8.1 (G), R50.1
- net MUX_PR1: now also R24.1; no longer Q8.1 (G), R50.1
- net PGND: now also R24.2, U4.2 (GND)
- net USB3V3: now also U4.3 (VO)
- net USB_VBUS: now also U4.1 (VI)
- net CHG_LATCH renamed MCU_CHG_BASE
- no-connect marks 24 -> 21
