File: hardware/v4/ups_v4/ups12v_v4.kicad_sch (KiCad schematic)
At the start: 124 parts, among them IC1 BQ25798RQMR, J1 ADAPTER 4.75-21V, J2 VSYS OUTPUT, J3 BATTERY 2S/4S, J4 MCU / BIAS INTERFACE, J6 NTC temp sensor, J7 USB-C PROGRAM / NATIVE USB, Q1 AON7528, Q2 AON7528, Q3 PMV16UN, Q4 BC847 INT DOMAIN ISOLATOR, Q5 BC857 MAIN-GATED CHG SOURCE, Q6 BC847 MAIN_VALID SINK, Q7 BC847 MCU CHG ARM SINK, Q8 PMV16UN MAIN_VALID, Q9 PMV16UN TCA_EN, SW1 BOOT / DOWNLOAD, SW2 RESET, U1 ESP32-C3-MINI-1-N4X, U2 TPD2EUSB30A (PROVISIONAL), U3 TPS62933DRLR NORMAL 3V3, U4 AP7361C-33E-13 USB 3V3 LDO, U5 TPS2116DRL NORMAL PRIORITY, U6 TCA9517DGKR REV.D

Commit message: phase 3.5
Other:
- note added: "CE pull-up via REGN/MAIN diode OR. BQ25792 2S charger-only reset/default 2A risk OPEN."
- note added: "CHARGING: MAIN PRESENT AND FIRMWARE REQUEST"
- note added: "Complete power interruption: EN 10k/1u RC and GPIO straps restart MCU. Transition resets acceptable; hardware tests pending."
- note added: "I2C / INT DOMAIN ISOLATION"
- note added: "NORMAL 3V3 / SERVICE USB 3V3"
- note added: "Optional independent 5V F5 block is NOT IMPLEMENTED; resolve F0-only versus common-PCB F5 before PCB freeze."
- note added: "POWER MUX - MAIN PRIORITY"
- note added: "Q5/Q6/Q7 default off; Q3 sinks CE only on request. Q6 is not a precision MAIN voltage monitor."
- note added: "SERVICE USB / ESP32-C3 RECOVERY - prototype, not fabrication approval"
- note added: "U1 project footprint corrected to 61 lands / 53 numbers; verify RF keepout, stencil and placement in PCB phase."
- note added: "U3 SYS -> MAIN_3V3 buck; U4 USB_VBUS -> USB3V3 LDO; U5 normal-priority mux -> MCU3V3."
- note added: "UPS V4 - complete prototype schematic / Phase 3.2 owner review"
- note added: "USB-only ROM flashing: BOOT held low during RESET; no battery/adapter required. Wi-Fi off in service firmware."
- note added: "VIN damping R12 2 ohm / C26 2.2uF 100V: selected prototype parts; VAC1 hot-plug qualification OPEN."
- note removed: "CE_N defaults OFF. MAIN_3V3 / CHG_REQ are the only intended control paths; USB 3V3 must not bias CE."
- note removed: "MCU3V3 is a reserved power-domain input; VSYS buck, USB buck and mux are pending next checkpoint."
- note removed: "PCB BLOCK: exact Espressif land-pattern comparison pending; readback is 62 physical pads / 60 unique numbers, duplicate ground numbers, no courtyard."
- note removed: "PHASE 3.1 CHECKPOINT: native USB / recovery wiring only"
- note removed: "TI Fig. 8-1 VIN damping: 2 ohm series plus 2.2 uF shunt to PGND; exact >=35 V parts pending procurement."
- note removed: "USB_VBUS is USB-only input; USB-derived 3V3 regulator is pending next checkpoint."
- note removed: "V4 Phase 2b charger / power stage - review checkpoint"
Changed lines of the file:
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@@
 		)
 	)
-	(text "TI Fig. 8-1 VIN damping: 2 ohm series plus 2.2 uF shunt to PGND; exact >=35 V parts pending procurement."
-		(at 24.13 41.91 0)
-		(effects
-			(font
-				(size 0.8 0.8)
-			)
-			(justify left bottom)
-		)
-	)
-	(text "CE_N defaults OFF. MAIN_3V3 / CHG_REQ are the only intended control paths; USB 3V3 must not bias CE."
-		(at 270.51 140.97 0)
-		(effects
-			(font
-				(size 1 1)
-				(bold yes)
-			)
-			(justify left bottom)
-		)
-	)
-	(text "V4 Phase 2b charger / power stage - review checkpoint"
-		(at 260.35 16.51 0)
-		(effects
-			(font
-				(size 1.27 1.27)
-				(bold yes)
-			)
-			(justify left bottom)
-		)
-	)
 	(text "PGND = system return; GND = quiet TS / PROG / NTC; NT1 local tie; no PCB moat."
 		(at 270.51 127 0)
@@
 		)
 	)
-	(text "PHASE 3.1 CHECKPOINT: native USB / recovery wiring only"
-		(at 225 275 0)
-		(effects
-			(font
-				(size 1.5 1.5)
-				(bold yes)
-			)
-			(justify left bottom)
-		)
-	)
-	(text "USB_VBUS is USB-only input; USB-derived 3V3 regulator is pending next checkpoint."
-		(at 225 278 0)
-		(effects
-			(font
-				(size 1.2 1.2)
-			)
-			(justify left bottom)
-		)
-	)
-	(text "MCU3V3 is a reserved power-domain input; VSYS buck, USB buck and mux are pending next checkpoint."
-		(at 225 281 0)
-		(effects
-			(font
-				(size 1.2 1.2)
-			)
-			(justify left bottom)
-		)
-	)
-	(text "PCB BLOCK: exact Espressif land-pattern comparison pending; readback is 62 physical pads / 60 unique numbers, duplicate ground numbers, no courtyard."
-		(at 225 284 0)
-		(effects
-			(font
-				(size 1.2 1.2)
-			)
-			(justify left bottom)
-		)
-	)
 	(label "NORMAL_EN"
 		(at 492.76 44.45 180)
@@
 		)
 	)
+  (text "UPS V4 - complete prototype schematic / Phase 3.2 owner review"
+    (at 260.35 16.51 0)
+    (effects (font (size 1.5 1.5) (bold yes)) (justify left bottom))
+  )
+  (text "VIN damping R12 2 ohm / C26 2.2uF 100V: selected prototype parts; VAC1 hot-plug qualification OPEN."
+    (at 24.13 41.91 0)
+    (effects (font (size 0.8 0.8)) (justify left bottom))
+  )
+  (text "SERVICE USB / ESP32-C3 RECOVERY - prototype, not fabrication approval"
+    (at 225 275 0)
+    (effects (font (size 1.5 1.5) (bold yes)) (justify left bottom))
+  )
+  (text "U3 SYS -> MAIN_3V3 buck; U4 USB_VBUS -> USB3V3 LDO; U5 normal-priority mux -> MCU3V3."
+    (at 225 279 0)
+    (effects (font (size 1.1 1.1)) (justify left bottom))
+  )
+  (text "USB-only ROM flashing: BOOT held low during RESET; no battery/adapter required. Wi-Fi off in service firmware."
+    (at 225 283 0)
+    (effects (font (size 1.1 1.1)) (justify left bottom))
+  )
+  (text "Complete power interruption: EN 10k/1u RC and GPIO straps restart MCU. Transition resets acceptable; hardware tests pending."
+    (at 225 287 0)
+    (effects (font (size 1.1 1.1)) (justify left bottom))
+  )
+  (text "U1 project footprint corrected to 61 lands / 53 numbers; verify RF keepout, stencil and placement in PCB phase."
+    (at 225 291 0)
+    (effects (font (size 1.1 1.1)) (justify left bottom))
+  )
+  (text "NORMAL 3V3 / SERVICE USB 3V3"
+    (at 470 28 0)
+    (effects (font (size 1.5 1.5) (bold yes)) (justify left bottom))
+  )
+  (text "POWER MUX - MAIN PRIORITY"
+    (at 575 81 0)
+    (effects (font (size 1.5 1.5) (bold yes)) (justify left bottom))
+  )
+  (text "I2C / INT DOMAIN ISOLATION"
+    (at 687 70 0)
+    (effects (font (size 1.5 1.5) (bold yes)) (justify left bottom))
+  )
+  (text "CHARGING: MAIN PRESENT AND FIRMWARE REQUEST"
+    (at 530 175 0)
+    (effects (font (size 1.5 1.5) (bold yes)) (justify left bottom))
+  )
+  (text "Q5/Q6/Q7 default off; Q3 sinks CE only on request. Q6 is not a precision MAIN voltage monitor."
+    (at 530 267 0)
+    (effects (font (size 1.1 1.1)) (justify left bottom))
+  )
+  (text "CE pull-up via REGN/MAIN diode OR. BQ25792 2S charger-only reset/default 2A risk OPEN."
+    (at 530 271 0)
+    (effects (font (size 1.1 1.1)) (justify left bottom))
+  )
+  (text "Optional independent 5V F5 block is NOT IMPLEMENTED; resolve F0-only versus common-PCB F5 before PCB freeze."
+    (at 225 300 0)
+    (effects (font (size 1.1 1.1)) (justify left bottom))
+  )
 	(symbol
 		(lib_id "Device:NetTie_2")
@@
 		(dnp no)
 		(property "Reference" "U2"
-			(at 309.88 208.28 0)
+			(at 309.88 205.55 0)
 			(effects
 				(font
@@
 		)
 		(property "Value" "TPD2EUSB30A (PROVISIONAL)"
-			(at 317.5 222.25 0)
+			(at 309.88 229.79 0)
 			(effects
 				(font
@@
 		(dnp no)
 		(property "Reference" "U5"
-			(at 591.566 86.106 0)
+			(at 599.44 83.63 0)
 			(effects
 				(font
@@
 		)
 		(property "Value" "TPS2116DRL NORMAL PRIORITY"
-			(at 599.948 104.14 0)
+			(at 599.44 110.41 0)
 			(effects
 				(font
@@
 		(dnp no)
 		(property "Reference" "U6"
-			(at 689.61 83.82 0)
+			(at 699.77 78.55 0)
 			(effects
 				(font
@@
 		)
 		(property "Value" "TCA9517DGKR REV.D"
-			(at 701.04 106.68 0)
+			(at 699.77 112.95 0)
 			(effects
 				(font
@@
 		(dnp no)
 		(property "Reference" "Q4"
-			(at 624.84 183.515 0)
+			(at 619.76 176.34 0)
 			(effects
 				(font
@@
 		)
 		(property "Value" "BC847 INT DOMAIN ISOLATOR"
-			(at 624.84 185.42 0)
+			(at 619.76 195.5 0)
 			(effects
 				(font
@@
 		(dnp no)
 		(property "Reference" "U3"
-			(at 500.38 35.56 0)
+			(at 500.38 35.37 0)
 			(effects
 				(font
@@
 		)
 		(property "Value" "TPS62933DRLR NORMAL 3V3"
-			(at 500.38 38.1 0)
+			(at 500.38 67.23 0)
 			(effects
 				(font
@@
 		(dnp no)
 		(property "Reference" "Q5"
-			(at 544.83 217.805 0)
+			(at 539.75 210.63 0)
 			(effects
 				(font
@@
 		)
 		(property "Value" "BC857 MAIN-GATED CHG SOURCE"
-			(at 544.83 219.71 0)
+			(at 539.75 229.79 0)
 			(effects
 				(font
@@
 		(dnp no)
 		(property "Reference" "Q6"
-			(at 604.52 202.565 0)
+			(at 599.44 195.39 0)
 			(effects
 				(font
@@
 		)
 		(property "Value" "BC847 MAIN_VALID SINK"
-			(at 604.52 204.47 0)
+			(at 599.44 214.55 0)
 			(effects
 				(font
@@
 		(dnp no)
 		(property "Reference" "Q7"
-			(at 684.53 202.565 0)
+			(at 679.45 195.39 0)
 			(effects
 				(font
@@
 		)
 		(property "Value" "BC847 MCU CHG ARM SINK"
-			(at 684.53 204.47 0)
+			(at 679.45 214.55 0)
 			(effects
 				(font
@@
 		(dnp no)
 		(property "Reference" "Q8"
-			(at 774.7 93.345 0)
+			(at 769.62 86.17 0)
 			(effects
 				(font
@@
 		)
 		(property "Value" "PMV16UN MAIN_VALID"
-			(at 774.7 95.25 0)
+			(at 769.62 105.33 0)
 			(effects
 				(font
@@
 		(dnp no)
 		(property "Reference" "Q9"
-			(at 774.7 118.745 0)
+			(at 769.62 111.57 0)
 			(effects
 				(font
@@
 		)
 		(property "Value" "PMV16UN TCA_EN"
-			(at 774.7 120.65 0)
+			(at 769.62 130.73 0)
 			(effects
 				(font
@@
 		(dnp no)
 		(property "Reference" "U4"
-			(at 496.57 141.605 0)
+			(at 500.38 138.875 0)
 			(effects
 				(font
@@
 		)
 		(property "Value" "AP7361C-33E-13 USB 3V3 LDO"
-			(at 500.38 141.605 0)
+			(at 500.38 157.4 0)
 			(effects
 				(font

Commit message: phase 3.7
Parts:
- added C60, C61: 10u/50V, Capacitor_SMD:C_1210_3225Metric, symbol Device:C
- added C62, C66, C67, C68, C69: 100n/50V, Capacitor_SMD:C_0603_1608Metric, symbol Device:C
- added C63: 33n/50V, Capacitor_SMD:C_0603_1608Metric, symbol Device:C
- added C64, C65: 22u/35V, Capacitor_SMD:C_1206_3216Metric, symbol Device:C
- added J8: 5V / GND, Connector_Phoenix_MSTB:PhoenixContact_MSTBA_2,5_2-G-5,08_1x02_P5.08mm_Horizontal, symbol Connector:Conn_01x02_Pin
- added L3: 6.8uH, Inductor_SMD:L_Coilcraft_XAL5050-XXX, symbol Device:L
- added Q10: AON7528, easyeda2kicad:DFN-8_L3.3-W3.3-P0.65-BL-3, symbol easyeda2kicad:AON7528_michal
- added R60: 53k 0.1%, Resistor_SMD:R_0603_1608Metric, symbol Device:R
- added R61: 10k 0.1%, Resistor_SMD:R_0603_1608Metric, symbol Device:R
- added R62: 100k 1%, Resistor_SMD:R_0603_1608Metric, symbol Device:R
- added R63: 38k3 1%, Resistor_SMD:R_0603_1608Metric, symbol Device:R
- added TP13: MAIN_3V3, TestPoint:TestPoint_Pad_D1.5mm, symbol Connector:TestPoint
- added TP14: CE_N, TestPoint:TestPoint_Pad_D1.5mm, symbol Connector:TestPoint
- added TP15: VIN1, TestPoint:TestPoint_Pad_D1.5mm, symbol Connector:TestPoint
- added TP16: BATTERY, TestPoint:TestPoint_Pad_D1.5mm, symbol Connector:TestPoint
- added TP17: F5_5V_OUT, TestPoint:TestPoint_Pad_D1.5mm, symbol Connector:TestPoint
- added TP5: ESP_TX (GPIO21), TestPoint:TestPoint_Pad_D1.5mm, symbol Connector:TestPoint
- added TP6: ESP_RX (GPIO20), TestPoint:TestPoint_Pad_D1.5mm, symbol Connector:TestPoint
- added TP7: PGND, TestPoint:TestPoint_Pad_D1.5mm, symbol Connector:TestPoint
- added TP8: MCU3V3, TestPoint:TestPoint_Pad_D1.5mm, symbol Connector:TestPoint
- added U7: TPS62933DRLR, Package_TO_SOT_SMD:SOT-583-8, symbol Regulator_Switching:TPS62933
- added U8: LM74700QDBVRQ1, Package_TO_SOT_SMD:SOT-23-6, symbol Power_Management:LM74700
- C33: value 22u NORMAL OUT -> 22u/35V NORMAL OUT; footprint Capacitor_SMD:C_0805_2012Metric -> Capacitor_SMD:C_1206_3216Metric; LCSC Part (none) -> C69612; MPN OPEN -> C3216X5R1V226M160AC; Manufacturer OPEN -> TDK; Parameters Prototype value candidate; exact MPN/supplier and temperatu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 -> Normal-output tolerance budget: 2x22uF pair; 25uF Ceff desi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; Source Ordinary passive; supplier verification deferred to BOM fre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 -> https://www.tme.eu/gb/details/c3216x5r1v226mac/mlcc-smd-cap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
- C45: value 22u NORMAL OUT 2 -> 22u/35V NORMAL OUT; footprint Capacitor_SMD:C_0805_2012Metric -> Capacitor_SMD:C_1206_3216Metric; ApprovalStatus (none) -> PROPOSED; LCSC Part (none) -> C69612; MPN (none) -> C3216X5R1V226M160AC; Manufacturer (none) -> TDK; Parameters (none) -> Normal-output tolerance budget: 2x22uF pair; 25uF Ceff desi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; Source (none) -> https://www.tme.eu/gb/details/c3216x5r1v226mac/mlcc-smd-cap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
- NT1, NT2, NT4: value ~ -> (none)
- R32: value 32k2 0.1% NORMAL FB -> 31k6 0.1% 10ppm NORMAL FB; ApprovalStatus (none) -> PROPOSED; MPN (none) -> RN73C1E31K6BTD; Manufacturer (none) -> TE Connectivity; Parameters (none) -> 0.1% 10ppm/K 0402 candidate; procurement open; owner author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
- R33: ApprovalStatus (none) -> PROPOSED; MPN (none) -> RN73C1E10KBTD; Manufacturer (none) -> TE Connectivity; Parameters (none) -> 10k 0.1% 10ppm/K maximum; procurement open; value and footp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
Connections:
- net BATTERY: now also TP16.1
- net CE_N: now also TP14.1
- net MAIN_3V3: now also TP13.1
- net MCU3V3: now also TP8.1
- net PGND: now also C60.2, C61.2, C63.2, C64.2, C65.2, C66.2, C68.2, C69.2, J8.2 (Pin_2), R61.2, R63.2, TP7.1, U7.4 (GND), U8.2 (GND)
- net SYS: now also C60.1, C61.1, C69.1, R62.1, U7.3 (VIN)
- net UART_RX: now also TP6.1
- net UART_TX: now also TP5.1
- net VIN1: now also TP15.1
- new net F5_5V_OUT: C68.1, J8.1 (Pin_1), Q10.5 (D), Q10.6 (D), Q10.7 (D), Q10.8 (D), Q10.9 (D), TP17.1, U8.4 (CATHODE)
- new net F5_BST: C62.1, U7.6 (BST)
- new net F5_EN: R62.2, R63.1, U7.2 (EN)
- new net F5_FB: R60.2, R61.1, U7.8 (FB)
- new net F5_GATE: Q10.4 (G), U8.5 (GATE)
- new net F5_RAW: C64.1, C65.1, C66.1, C67.2, L3.2, Q10.1 (S), Q10.2 (S), Q10.3 (S), R60.1, U8.3 (EN), U8.6 (ANODE)
- new net F5_SS: C63.1, U7.7 (SS)
- new net F5_SW: C62.2, L3.1, U7.5 (SW)
- new net F5_VCAP: C67.1, U8.1 (VCAP)
- no-connect marks 21 -> 22
Other:
- note added: "F5 OPTIONAL 5V / 2A: populate ALL U7 U8 Q10 L3 R60-R63 C60-C69 J8; F0 omit all."
- note added: "OPTIONAL EMERGENCY UART: TP5 ESP_TX GPIO21, TP6 ESP_RX GPIO20, TP7 GND; no fitted header."
- note added: "PCB edge, 2.54mm pitch TOP view; triangle at TP5. UART high-Z while target off; NO power input."
- note added: "POWER MEASUREMENTS: TP15 VIN1, TP16 BATTERY, existing TP4 SYS; separate from MCU pogo group."
- note added: "PRIMARY SERVICE: native USB-C Serial/JTAG for programming, logging and debug; USB-only MCU power."
- note added: "SEPARATE MEASUREMENT ONLY: TP8 MCU3V3, TP13 MAIN_3V3; NOT in UART group. BOOT/RESET buttons retained."
- note added: "SYS 6-18V -> 5.04V buck -> ideal diode -> J8 pin1 +5V, pin2 PGND. No MCU/USB control."
- note added: "TP14 CE_N: separate passive charger-domain bring-up probe. No added RESET/BOOT/I2C pads."
- note added: "TP17 F5 OUTPUT: measurement only. No testpad is an authorized power input."
- note removed: "Optional independent 5V F5 block is NOT IMPLEMENTED; resolve F0-only versus common-PCB F5 before PCB freeze."
- note removed: "UPS V4 - complete prototype schematic / Phase 3.2 owner review"

Commit message: phase 4.3
Parts:
- J4: footprint Connector_JST:JST_XH_B6B-XH-A_1x06_P2.50mm_Vertical -> Connector_JST:JST_XH_S6B-XH-A_1x06_P2.50mm_Horizontal
- J6: footprint Connector_JST:JST_XH_B2B-XH-A_1x02_P2.50mm_Vertical -> Connector_JST:JST_XH_S2B-XH-A-1_1x02_P2.50mm_Horizontal
Changed lines of the file:
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@@
 			)
 		)
-		(property "Footprint" "Connector_JST:JST_XH_B2B-XH-A_1x02_P2.50mm_Vertical"
+		(property "Footprint" "Connector_JST:JST_XH_S2B-XH-A-1_1x02_P2.50mm_Horizontal"
 			(at 127 160.02 0)
 			(hide yes)
@@
 			)
 		)
-		(property "Footprint" "Connector_JST:JST_XH_B6B-XH-A_1x06_P2.50mm_Vertical"
+		(property "Footprint" "Connector_JST:JST_XH_S6B-XH-A_1x06_P2.50mm_Horizontal"
 			(at 96.52 118.11 0)
 			(hide yes)
