File: hardware/v4/ups_v4/ups12v_v4.kicad_sch (KiCad schematic)
At the start: 152 parts, among them IC1 BQ25798RQMR, J1 ADAPTER 4.75-21V, J2 VSYS OUTPUT, J3 BATTERY 2S/4S, J4 MCU / BIAS INTERFACE, J6 NTC temp sensor, J7 USB-C PROGRAM / NATIVE USB, J8 5V / GND, Q1 AON7528, Q10 AON7528, Q2 AON7528, Q3 PMV16UN, Q4 BC847 INT DOMAIN ISOLATOR, Q5 BC857 MAIN-GATED CHG SOURCE, Q6 BC847 MAIN_VALID SINK, Q7 BC847 MCU CHG ARM SINK, Q8 PMV16UN MAIN_VALID, Q9 PMV16UN TCA_EN, SW1 BOOT / DOWNLOAD, SW2 RESET, U1 ESP32-C3-MINI-1-N4X, U2 TPD2EUSB30A (PROVISIONAL), U3 TPS62933DRLR NORMAL 3V3, U4 AP7361C-33E-13 USB 3V3 LDO, U5 TPS2116DRL NORMAL PRIORITY, U6 TCA9517DGKR REV.D, U7 TPS62933DRLR, U8 LM74700QDBVRQ1

Commit message: phase 4.4
Parts:
- added C70, C71: 1u 16V X7R, Capacitor_SMD:C_0603_1608Metric, symbol Device:C
- J7: footprint Connector_USB:USB_C_Receptacle_GCT_USB4105-xx-A_16P_TopMnt_Horizontal -> Connector_USB:USB_C_Receptacle_GCT_USB4085; ApprovalStatus PROPOSED -> APPROVED; LCSC (none) -> C7095263; MPN OPEN -> USB4085-GF-A; Manufacturer OPEN -> GCT; Parameters (none) -> USB2.0 16 THT contacts + 4 plated shell slots; preserve A/B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; Source Exact connector MPN/footprint pending verification -> Owner Phase 4.4 approval; GCT USB4085 Rev B 2023-02-28 shee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
Connections:
- net MAIN_3V3: now also C70.1
- net PGND: now also C70.2, C71.2
- net USB3V3: now also C71.1

Commit message: nanofit
Parts:
- J1: footprint TerminalBlock_Phoenix:TerminalBlock_Phoenix_MKDS-1,5-2-5.08_1x02_P5.08mm_Horizontal -> ups_v4:Molex_Nano-Fit_105313-xx02_1x02_P2.50mm_Horizontal_RevJ1; symbol My Connectors:Screw_Terminal_01x02 -> Connector_Generic:Conn_01x02; ApprovalStatus (none) -> APPROVED for CAD; MPN (none) -> 1053131102; Manufacturer (none) -> Molex; Parameters (none) -> Mating 1053071202; 1053002100 tin terminals; 1=PGND; 2=adap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; VerificationDate (none) -> 2026-10-11
- J2: footprint TerminalBlock_Phoenix:TerminalBlock_Phoenix_MKDS-1,5-2-5.08_1x02_P5.08mm_Horizontal -> ups_v4:Molex_Nano-Fit_105313-xx03_1x03_P2.50mm_Horizontal_RevJ1; symbol My Connectors:Screw_Terminal_01x02 -> Connector_Generic:Conn_01x03; ApprovalStatus (none) -> APPROVED for CAD; LCSC Part (none) -> C561764; MPN (none) -> 1053131103; Manufacturer (none) -> Molex; Parameters (none) -> Mating 1053071203; 1053002100 tin terminals; 1=PGND; 3=SYS;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; VerificationDate (none) -> 2026-10-11
- J3: footprint TerminalBlock_Phoenix:TerminalBlock_Phoenix_MKDS-1,5-2-5.08_1x02_P5.08mm_Horizontal -> ups_v4:Molex_Nano-Fit_105313-xx02_1x02_P2.50mm_Horizontal_RevJ1; symbol My Connectors:Screw_Terminal_01x02 -> Connector_Generic:Conn_01x02; ApprovalStatus (none) -> APPROVED for CAD; LCSC Part (none) -> C17189968; MPN (none) -> 1053132102; Manufacturer (none) -> Molex; Parameters (none) -> Mating 1053072202; 1053002100 tin terminals; 1=PGND; 2=BATT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; VerificationDate (none) -> 2026-10-11
- J8: footprint Connector_Phoenix_MSTB:PhoenixContact_MSTBA_2,5_2-G-5,08_1x02_P5.08mm_Horizontal -> ups_v4:Molex_Nano-Fit_105313-xx03_1x03_P2.50mm_Horizontal_RevJ1; symbol Connector:Conn_01x02_Pin -> Connector:Conn_01x03_Pin; ApprovalStatus PROPOSED -> APPROVED for CAD; MPN 1757242 -> 1053132103; Manufacturer Phoenix Contact -> Molex; Parameters MSTBA 2,5/2-G-5,08;12A rated;1=5V2=PGND; mating1757019 cand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 -> Mating 1053072203; 1053002100 tin terminals; 1=PGND; 3=F5_5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; VerificationDate 2026-10-10 -> 2026-10-11
Connections:
- net F5_5V_OUT: now also J8.3 (Pin_3); no longer J8.1 (Pin_1)
- net PGND: now also J8.1 (Pin_1); no longer J8.2 (Pin_2)
- net SYS: now also J2.3 (Pin_3); no longer J2.2 (Pin_2)
- no-connect marks 22 -> 24
Changed lines of the file:
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@@
 		(diameter 0)
 	)
-	(junction
-		(at 410.21 535.94)
-		(diameter 0)
-	)
 	(no_connect
 		(at 346.71 78.74)
@@
 		(at 203.2 474.98)
 	)
+	(no_connect
+		(at 116.84 29.21)
+	)
+	(no_connect
+		(at 415.29 477.52)
+	)
 	(wire
 		(pts
@@
 	(wire
 		(pts
-			(xy 116.84 29.21)
-			(xy 119.38 29.21)
-		)
-		(stroke
-			(width 0)
-			(type default)
-		)
-	)
-	(wire
-		(pts
 			(xy 346.71 119.38)
 			(xy 344.17 119.38)
@@
 	(wire
 		(pts
-			(xy 400.05 477.52)
-			(xy 415.29 477.52)
-		)
-	)
-	(wire
-		(pts
 			(xy 391.16 480.06)
 			(xy 391.16 488.95)
@@
 	(wire
 		(pts
-			(xy 415.29 474.98)
-			(xy 410.21 474.98)
-		)
-	)
-	(wire
-		(pts
-			(xy 410.21 474.98)
-			(xy 410.21 535.94)
-		)
-	)
-	(wire
-		(pts
 			(xy 110.49 535.94)
 			(xy 410.21 535.94)
@@
 		)
 	)
+	(wire
+		(pts
+			(xy 119.38 29.21)
+			(xy 119.38 31.75)
+		)
+	)
+	(wire
+		(pts
+			(xy 119.38 31.75)
+			(xy 116.84 31.75)
+		)
+	)
+	(wire
+		(pts
+			(xy 410.21 480.06)
+			(xy 415.29 480.06)
+		)
+	)
+	(wire
+		(pts
+			(xy 400.05 477.52)
+			(xy 400.05 474.98)
+		)
+	)
+	(wire
+		(pts
+			(xy 400.05 474.98)
+			(xy 415.29 474.98)
+		)
+	)
+	(wire
+		(pts
+			(xy 410.21 480.06)
+			(xy 410.21 535.94)
+		)
+	)
 	(text "USB-only ROM flashing: BOOT held low during RESET; no battery/adapter required. Wi-Fi off in service firmware."
 		(at 225 283 0)
@@
 	)
 	(label "F5_5V_OUT"
-		(at 415.29 477.52 180)
+		(at 187.96 408.94 0)
 		(effects
 			(font
 				(size 1.27 1.27)
 			)
-			(justify right bottom)
+			(justify left bottom)
 		)
 	)
 	(label "F5_5V_OUT"
-		(at 187.96 408.94 0)
+		(at 415.29 474.98 180)
 		(effects
 			(font
 				(size 1.27 1.27)
 			)
-			(justify left bottom)
+			(justify right bottom)
 		)
 	)
@@
 	)
 	(symbol
-		(lib_id "My Connectors:Screw_Terminal_01x02")
+		(lib_id "Connector_Generic:Conn_01x03")
 		(at 111.76 29.21 180)
 		(unit 1)
@@
 			)
 		)
-		(property "Footprint" "TerminalBlock_Phoenix:TerminalBlock_Phoenix_MKDS-1,5-2-5.08_1x02_P5.08mm_Horizontal"
+		(property "Footprint" "ups_v4:Molex_Nano-Fit_105313-xx03_1x03_P2.50mm_Horizontal_RevJ1"
 			(at 111.76 37.084 0)
 			(hide yes)
@@
 			)
 		)
-		(property "Datasheet" ""
+		(property "Datasheet" "https://www.molex.com/content/dam/molex/molex-dot-com/products/automated/en-us/salesdrawingpdf/105/105313/1053131102_sd.pdf"
 			(at 111.76 29.21 0)
 			(hide yes)
@@
 			)
 		)
-		(property "Description" "Generic screw terminal, single row, 01x02, script generated (kicad-library-utils/schlib/autogen/connector/)"
+		(property "Description" "Molex Nano-Fit 3-position right-angle through-hole header, key A, tin"
 			(at 112.776 34.544 0)
 			(hide yes)
@@
 			)
 		)
-		(property "Parameters" ""
+		(property "Parameters" "Mating 1053071203; 1053002100 tin terminals; 1=PGND; 3=SYS; 2=NC, uncrimped; Rev J1 NPTH pattern"
 			(at 111.76 29.21 0)
 			(hide yes)
@@
 			)
 		)
-		(property "LCSC Part" ""
+		(property "LCSC Part" "C561764"
 			(at 111.76 29.21 0)
 			(hide yes)
@@
 			)
 		)
-	)
+		(property "ApprovalStatus" "APPROVED for CAD"
+			(at 111.76 29.21 0)
+			(hide yes)
+			(effects
+				(font
+					(size 1.27 1.27)
+				)
+			)
+		)
+		(property "MPN" "1053131103"
+			(at 111.76 29.21 0)
+			(hide yes)
+			(effects
+				(font
+					(size 1.27 1.27)
+				)
+			)
+		)
+		(property "Manufacturer" "Molex"
+			(at 111.76 29.21 0)
+			(hide yes)
+			(effects
+				(font
+					(size 1.27 1.27)
+				)
+			)
+		)
+		(property "VerificationDate" "2026-10-11"
+			(at 111.76 29.21 0)
+			(hide yes)
+			(effects
+				(font
+					(size 1.27 1.27)
+				)
+			)
+		))
 	(symbol
 		(lib_id "Device:R")
@@
 	)
 	(symbol
-		(lib_id "My Connectors:Screw_Terminal_01x02")
+		(lib_id "Connector_Generic:Conn_01x02")
 		(at 73.66 29.21 180)
 		(unit 1)
@@
 			)
 		)
-		(property "Footprint" "TerminalBlock_Phoenix:TerminalBlock_Phoenix_MKDS-1,5-2-5.08_1x02_P5.08mm_Horizontal"
+		(property "Footprint" "ups_v4:Molex_Nano-Fit_105313-xx02_1x02_P2.50mm_Horizontal_RevJ1"
 			(at 73.66 37.084 0)
 			(hide yes)
@@
 			)
 		)
-		(property "Datasheet" ""
+		(property "Datasheet" "https://www.molex.com/content/dam/molex/molex-dot-com/products/automated/en-us/salesdrawingpdf/105/105313/1053131102_sd.pdf"
 			(at 73.66 29.21 0)
 			(hide yes)
@@
 			)
 		)
-		(property "Description" "Generic screw terminal, single row, 01x02, script generated (kicad-library-utils/schlib/autogen/connector/)"
+		(property "Description" "Molex Nano-Fit 2-position right-angle through-hole header, key B, tin"
 			(at 74.676 34.544 0)
 			(hide yes)
@@
 			)
 		)
-		(property "Parameters" ""
+		(property "Parameters" "Mating 1053072202; 1053002100 tin terminals; 1=PGND; 2=BATTERY; Rev J1 NPTH pattern"
 			(at 73.66 29.21 0)
 			(hide yes)
@@
 			)
 		)
-		(property "LCSC Part" ""
+		(property "LCSC Part" "C17189968"
 			(at 73.66 29.21 0)
 			(hide yes)
@@
 			)
 		)
-	)
+		(property "ApprovalStatus" "APPROVED for CAD"
+			(at 73.66 29.21 0)
+			(hide yes)
+			(effects
+				(font
+					(size 1.27 1.27)
+				)
+			)
+		)
+		(property "MPN" "1053132102"
+			(at 73.66 29.21 0)
+			(hide yes)
+			(effects
+				(font
+					(size 1.27 1.27)
+				)
+			)
+		)
+		(property "Manufacturer" "Molex"
+			(at 73.66 29.21 0)
+			(hide yes)
+			(effects
+				(font
+					(size 1.27 1.27)
+				)
+			)
+		)
+		(property "VerificationDate" "2026-10-11"
+			(at 73.66 29.21 0)
+			(hide yes)
+			(effects
+				(font
+					(size 1.27 1.27)
+				)
+			)
+		))
 	(symbol
 		(lib_id "Mechanical:MountingHole")
@@
 	)
 	(symbol
-		(lib_id "My Connectors:Screw_Terminal_01x02")
+		(lib_id "Connector_Generic:Conn_01x02")
 		(at 45.72 29.21 0)
 		(mirror x)
@@
 			)
 		)
-		(property "Footprint" "TerminalBlock_Phoenix:TerminalBlock_Phoenix_MKDS-1,5-2-5.08_1x02_P5.08mm_Horizontal"
+		(property "Footprint" "ups_v4:Molex_Nano-Fit_105313-xx02_1x02_P2.50mm_Horizontal_RevJ1"
 			(at 45.72 37.084 0)
 			(hide yes)
@@
 			)
 		)
-		(property "Datasheet" ""
+		(property "Datasheet" "https://www.molex.com/content/dam/molex/molex-dot-com/products/automated/en-us/salesdrawingpdf/105/105313/1053131102_sd.pdf"
 			(at 45.72 29.21 0)
 			(hide yes)
@@
 			)
 		)
-		(property "Description" "Generic screw terminal, single row, 01x02, script generated (kicad-library-utils/schlib/autogen/connector/)"
+		(property "Description" "Molex Nano-Fit 2-position right-angle through-hole header, key A, tin"
 			(at 44.704 34.544 0)
 			(hide yes)
@@
 			)
 		)
-		(property "Parameters" ""
+		(property "Parameters" "Mating 1053071202; 1053002100 tin terminals; 1=PGND; 2=adapter positive; Rev J1 NPTH pattern"
 			(at 45.72 29.21 0)
 			(hide yes)
@@
 			)
 		)
-	)
+		(property "ApprovalStatus" "APPROVED for CAD"
+			(at 45.72 29.21 0)
+			(hide yes)
+			(effects
+				(font
+					(size 1.27 1.27)
+				)
+			)
+		)
+		(property "MPN" "1053131102"
+			(at 45.72 29.21 0)
+			(hide yes)
+			(effects
+				(font
+					(size 1.27 1.27)
+				)
+			)
+		)
+		(property "Manufacturer" "Molex"
+			(at 45.72 29.21 0)
+			(hide yes)
+			(effects
+				(font
+					(size 1.27 1.27)
+				)
+			)
+		)
+		(property "VerificationDate" "2026-10-11"
+			(at 45.72 29.21 0)
+			(hide yes)
+			(effects
+				(font
+					(size 1.27 1.27)
+				)
+			)
+		))
 	(symbol
 		(lib_id "ups_v4_custom:ESP32-C3-MINI-1")
@@
 	)
 	(symbol
-		(lib_id "Connector:Conn_01x02_Pin")
+		(lib_id "Connector:Conn_01x03_Pin")
 		(at 420.37 477.52 180)
 		(unit 1)
@@
 			)
 		)
-		(property "Footprint" "Connector_Phoenix_MSTB:PhoenixContact_MSTBA_2,5_2-G-5,08_1x02_P5.08mm_Horizontal"
+		(property "Footprint" "ups_v4:Molex_Nano-Fit_105313-xx03_1x03_P2.50mm_Horizontal_RevJ1"
 			(at 420.37 477.52 0)
 			(hide yes)
@@
 			)
 		)
-		(property "Datasheet" ""
+		(property "Datasheet" "https://www.molex.com/content/dam/molex/molex-dot-com/products/automated/en-us/salesdrawingpdf/105/105313/1053131102_sd.pdf"
 			(at 420.37 477.52 0)
 			(hide yes)
@@
 			)
 		)
-		(property "Description" "Generic connector, single row, 01x02, script generated"
+		(property "Description" "Molex Nano-Fit 3-position right-angle through-hole header, key B, tin"
 			(at 420.37 477.52 0)
 			(hide yes)
@@
 			)
 		)
-		(property "ApprovalStatus" "PROPOSED"
+		(property "ApprovalStatus" "APPROVED for CAD"
 			(at 420.37 477.52 0)
 			(hide yes)
@@
 			)
 		)
-		(property "MPN" "1757242"
+		(property "MPN" "1053132103"
 			(at 420.37 477.52 0)
 			(hide yes)
@@
 			)
 		)
-		(property "Manufacturer" "Phoenix Contact"
+		(property "Manufacturer" "Molex"
 			(at 420.37 477.52 0)
 			(hide yes)
@@
 			)
 		)
-		(property "Parameters" "MSTBA 2,5/2-G-5,08;12A rated;1=5V2=PGND; mating1757019 candidate verify harness beforefreeze"
+		(property "Parameters" "Mating 1053072203; 1053002100 tin terminals; 1=PGND; 3=F5_5V_OUT; 2=NC, uncrimped; Rev J1 NPTH pattern"
 			(at 420.37 477.52 0)
 			(hide yes)
@@
 			)
 		)
-		(property "VerificationDate" "2026-10-10"
+		(property "VerificationDate" "2026-10-11"
 			(at 420.37 477.52 0)
 			(hide yes)
@@
 			)
 		)
-	)
+		(property "LCSC Part" ""
+			(at 420.37 477.52 0)
+			(hide yes)
+			(effects
+				(font
+					(size 1.27 1.27)
+				)
+			)
+		))
 	(symbol
 		(lib_id "power:PWR_FLAG")

Commit message: phase 4.13
Connections:
- net USB_MCU_DN: now reaches R49.1, U1.26 (USB_D-_/_GPIO18)
- net USB_MCU_DP: now reaches R48.1, U1.27 (USB_D+_/_GPIO19)
Changed lines of the file:
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@@
 		)
 	)
+	(label "USB_MCU_DP"
+		(at 436.88 134.62 0)
+		(effects
+			(font
+				(size 1.27 1.27)
+			)
+			(justify left bottom)
+		)
+	)
+	(label "USB_MCU_DN"
+		(at 436.88 132.08 0)
+		(effects
+			(font
+				(size 1.27 1.27)
+			)
+			(justify left bottom)
+		)
+	)
 	(global_label "PGND"
 		(shape input)
@@
 			)
 		)
-		(body_style 1)
-		(in_pos_files yes)
-		(pin "1"
-		)
-		(pin "2"
-		)
-		(instances
-			(project "ups12v_v4"
-				(path "/ce327fff-9e65-43e6-a970-97add7a9f6f7"
-					(reference "J2")
-					(unit 1)
-				)
-			)
-		)
 		(property "ApprovalStatus" "APPROVED for CAD"
 			(at 111.76 29.21 0)
@@
 				)
 			)
-		))
+		)
+		(body_style 1)
+		(in_pos_files yes)
+		(pin "1"
+		)
+		(pin "2"
+		)
+		(instances
+			(project "ups12v_v4"
+				(path "/ce327fff-9e65-43e6-a970-97add7a9f6f7"
+					(reference "J2")
+					(unit 1)
+				)
+			)
+		)
+	)
 	(symbol
 		(lib_id "Device:R")
@@
 			)
 		)
-		(body_style 1)
-		(in_pos_files yes)
-		(pin "1"
-		)
-		(pin "2"
-		)
-		(instances
-			(project "ups12v_v4"
-				(path "/ce327fff-9e65-43e6-a970-97add7a9f6f7"
-					(reference "J3")
-					(unit 1)
-				)
-			)
-		)
 		(property "ApprovalStatus" "APPROVED for CAD"
 			(at 73.66 29.21 0)
@@
 				)
 			)
-		))
+		)
+		(body_style 1)
+		(in_pos_files yes)
+		(pin "1"
+		)
+		(pin "2"
+		)
+		(instances
+			(project "ups12v_v4"
+				(path "/ce327fff-9e65-43e6-a970-97add7a9f6f7"
+					(reference "J3")
+					(unit 1)
+				)
+			)
+		)
+	)
 	(symbol
 		(lib_id "Mechanical:MountingHole")
@@
 			)
 		)
-		(body_style 1)
-		(in_pos_files yes)
-		(pin "1"
-		)
-		(pin "2"
-		)
-		(instances
-			(project "ups12v_v4"
-				(path "/ce327fff-9e65-43e6-a970-97add7a9f6f7"
-					(reference "J1")
-					(unit 1)
-				)
-			)
-		)
 		(property "ApprovalStatus" "APPROVED for CAD"
 			(at 45.72 29.21 0)
@@
 				)
 			)
-		))
+		)
+		(body_style 1)
+		(in_pos_files yes)
+		(pin "1"
+		)
+		(pin "2"
+		)
+		(instances
+			(project "ups12v_v4"
+				(path "/ce327fff-9e65-43e6-a970-97add7a9f6f7"
+					(reference "J1")
+					(unit 1)
+				)
+			)
+		)
+	)
 	(symbol
 		(lib_id "ups_v4_custom:ESP32-C3-MINI-1")
@@
 			)
 		)
-		(instances
-			(project "ups12v_v4"
-				(path "/ce327fff-9e65-43e6-a970-97add7a9f6f7"
-					(reference "J8")
-					(unit 1)
-				)
-			)
-		)
 		(property "LCSC Part" ""
 			(at 420.37 477.52 0)
@@
 				)
 			)
-		))
+		)
+		(instances
+			(project "ups12v_v4"
+				(path "/ce327fff-9e65-43e6-a970-97add7a9f6f7"
+					(reference "J8")
+					(unit 1)
+				)
+			)
+		)
+	)
 	(symbol
 		(lib_id "power:PWR_FLAG")
