File: hardware/v4/ups_v4/ups12v_v4.kicad_pcb (KiCad board)
At the start: 4 copper layers, 152 parts, among them IC1 BQ25798RQMR, J1 ADAPTER 4.75-21V, J2 VSYS OUTPUT, J3 BATTERY 2S/4S, J4 MCU / BIAS INTERFACE, J6 NTC temp sensor, J7 USB-C PROGRAM / NATIVE USB, J8 5V / GND, Q1 AON7528, Q10 AON7528, Q2 AON7528, Q3 PMV16UN, Q4 BC847 INT DOMAIN ISOLATOR, Q5 BC857 MAIN-GATED CHG SOURCE, Q6 BC847 MAIN_VALID SINK, Q7 BC847 MCU CHG ARM SINK, Q8 PMV16UN MAIN_VALID, Q9 PMV16UN TCA_EN, SW1 BOOT / DOWNLOAD, SW2 RESET, U1 ESP32-C3-MINI-1-N4X, U2 TPD2EUSB30A (PROVISIONAL), U3 TPS62933DRLR NORMAL 3V3, U4 AP7361C-33E-13 USB 3V3 LDO, U5 TPS2116DRL NORMAL PRIORITY, U6 TCA9517DGKR REV.D, U7 TPS62933DRLR, U8 LM74700QDBVRQ1

Commit message: phase 4.3
Parts:
- moved C68 97.1 mm to (116.5, 50.0), turned to 90 degrees
- moved C67 95.0 mm to (116.0, 53.0), turned to 90 degrees
- moved H4 93.8 mm to (121.0, 95.0)
- moved TP17 87.4 mm to (115.5, 44.5)
- moved C66 85.8 mm to (107.5, 54.5)
- moved C69 83.3 mm to (110.0, 54.0), turned to 90 degrees
- moved H2 83.3 mm to (121.0, 46.0)
- moved U4 81.8 mm to (109.0, 83.0)
- moved C63 81.3 mm to (105.0, 63.0)
- moved R60 78.3 mm to (105.0, 57.2), turned to 90 degrees
- moved R61 78.1 mm to (105.0, 60.4), turned to 90 degrees
- moved C62 76.0 mm to (99.7, 60.5), turned to 90 degrees
- moved U8 75.9 mm to (113.0, 53.0)
- moved U2 75.6 mm to (113.8, 78.5), turned to 90 degrees
- moved C27 74.2 mm to (115.5, 87.4)
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Other:
- board outline added: 96 x 70 mm
- board text added: ">"
- board text added: "GND"
- board text added: "RF: ALL LAYERS CLEAR - 15 mm EXTERNAL METAL CLEARANCE"
- board text added: "RX"
- board text added: "TX"

Commit message: phase 4.3
Parts:
- J4: footprint Connector_JST:JST_XH_B6B-XH-A_1x06_P2.50mm_Vertical -> Connector_JST:JST_XH_S6B-XH-A_1x06_P2.50mm_Horizontal
- J6: footprint Connector_JST:JST_XH_B2B-XH-A_1x02_P2.50mm_Vertical -> Connector_JST:JST_XH_S2B-XH-A-1_1x02_P2.50mm_Horizontal
- moved C30 19.7 mm to (91.0, 93.5)
- moved C31 17.9 mm to (90.0, 96.0)
- moved C3 17.5 mm to (56.3, 67.4), turned to -90 degrees
- moved C27 14.6 mm to (102.5, 80.7), turned to 180 degrees
- moved J4 4.00 mm to (122.5, 40.0)
- moved J6 2.50 mm to (104.0, 38.5)
- moved H1 1.50 mm to (35.0, 47.5)
- moved H2 1.50 mm to (121.0, 47.5)

Commit message: phase 4.4
Parts:
- added C70: 1u 16V X7R, Capacitor_SMD:C_0603_1608Metric, F.Cu at (62.8, 84.5)
- added C71: 1u 16V X7R, Capacitor_SMD:C_0603_1608Metric, F.Cu at (67.9, 82.8)
- J7: footprint Connector_USB:USB_C_Receptacle_GCT_USB4105-xx-A_16P_TopMnt_Horizontal -> Connector_USB:USB_C_Receptacle_GCT_USB4085
- moved J7 3.96 mm to (117.4, 84.0)
- moved C36 3.86 mm to (67.5, 80.0), turned to 90 degrees

Commit message: phase 4.5
Parts:
- moved C6 3.75 mm to (58.6, 62.8)
- moved C5 2.19 mm to (61.4, 62.8)
- moved Q3 1.74 mm to (77.8, 63.2), turned to 180 degrees
- moved C1 0.90 mm to (64.5, 65.0)
- turned C26 to 180 degrees
Routing:
- net VIN1: track 0.00 -> 87.1 mm, vias 0 -> 10
- net BATTERY: track 0.00 -> 77.1 mm, vias 0 -> 8
- net SYS: track 0.00 -> 68.3 mm, vias 0 -> 4
- net Net-(D1-K): track 0.00 -> 45.1 mm, vias 0 -> 4
- net VBUS: track 0.00 -> 35.3 mm, vias 0 -> 14
- net Net-(NT4-Pad2): track 0.00 -> 29.5 mm, vias 0 -> 7
- net SW2: track 0.00 -> 29.0 mm, vias 0 -> 19
- net SW1: track 0.00 -> 28.0 mm, vias 0 -> 19
- net PGND: track 0.00 -> 26.4 mm, vias 0 -> 42
- net ACDRV1: track 0.00 -> 15.5 mm, vias 0 -> 2
- net Net-(J1-Pin_2): track 0.00 -> 15.0 mm
- net PMID: track 0.00 -> 13.4 mm
- net Net-(D1-A): track 0.00 -> 12.1 mm
- net BTST2: track 0.00 -> 7.42 mm, vias 0 -> 2
- net Net-(C26-Pad1): track 0.00 -> 7.08 mm
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- added copper zone on In1.Cu, net PGND

Commit message: phase 4.6
Parts:
- moved C12 4.88 mm to (51.2, 55.0)
- moved C15 1.88 mm to (58.6, 60.6), turned to 0 degrees
- moved C17 1.80 mm to (63.7, 60.6)
- moved L1 1.70 mm to (60.0, 52.2)
- moved C14 1.25 mm to (65.8, 60.6)
- moved C11 0.55 mm to (68.0, 60.0)
Routing:
- net PMID: track 13.4 -> 19.5 mm
- net PGND: track 26.4 -> 31.8 mm, vias 42 -> 46
- net SW2: track 29.0 -> 26.9 mm
- net SYS: track 68.3 -> 69.5 mm
- net SW1: track 28.0 -> 26.9 mm

Commit message: nanofit
Parts:
- J1, J3: footprint TerminalBlock_Phoenix:TerminalBlock_Phoenix_MKDS-1,5-2-5.08_1x02_P5.08mm_Horizontal -> ups_v4:Molex_Nano-Fit_105313-xx02_1x02_P2.50mm_Horizontal_RevJ1
- J2: footprint TerminalBlock_Phoenix:TerminalBlock_Phoenix_MKDS-1,5-2-5.08_1x02_P5.08mm_Horizontal -> ups_v4:Molex_Nano-Fit_105313-xx03_1x03_P2.50mm_Horizontal_RevJ1
- J8: footprint Connector_Phoenix_MSTB:PhoenixContact_MSTBA_2,5_2-G-5,08_1x02_P5.08mm_Horizontal -> ups_v4:Molex_Nano-Fit_105313-xx03_1x03_P2.50mm_Horizontal_RevJ1
- moved J1 4.38 mm to (43.0, 40.4), turned to 90 degrees
- moved J2 4.38 mm to (58.0, 40.4), turned to 90 degrees
- moved J3 4.38 mm to (73.0, 40.4), turned to 90 degrees
- moved J8 0.62 mm to (89.0, 40.4), turned to 90 degrees
Connections:
- J2 pad 2: SYS -> unconnected-(J2-Pin_2-Pad2)
- J8 pad 1: /F5_5V_OUT -> PGND
- J8 pad 2: PGND -> unconnected-(J8-Pin_2-Pad2)
Routing:
- net BATTERY: track 77.1 -> 65.1 mm
- net Net-(J1-Pin_2): track 15.0 -> 3.85 mm
- net SYS: track 69.5 -> 75.2 mm

Commit message: recovery
Parts:
- moved C9 7.08 mm to (61.1, 69.1)
Routing:
- net VIN1: track 87.1 -> 78.4 mm, vias 10 -> 8
- net PGND: track 31.8 -> 30.0 mm, vias 46 -> 47
Changed lines of the file:
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@@
 		(duplicate_pad_numbers_are_jumpers no)
 		(fp_line
+			(start 10.03 -1.83)
+			(end 1.81 -1.83)
+			(stroke
+				(width 0.12)
+				(type default)
+			)
+			(layer "F.SilkS")
+		)
+		(fp_line
+			(start 1.81 -1.83)
+			(end 1.81 6.83)
+			(stroke
+				(width 0.12)
+				(type default)
+			)
+			(layer "F.SilkS")
+		)
+		(fp_line
 			(start 0.3 -1.534264)
 			(end -0.3 -1.534264)
@@
 			(layer "F.SilkS")
 		)
-		(fp_rect
-			(start 1.81 -1.83)
-			(end 10.49 6.83)
+		(fp_line
+			(start 1.81 6.83)
+			(end 10.03 6.83)
 			(stroke
 				(width 0.12)
-				(type solid)
+				(type default)
 			)
-			(fill no)
 			(layer "F.SilkS")
 		)
@@
 		(fp_line
 			(start 7.57 6)
-			(end 7.57 8.73)
+			(end 7.57 8.26)
 			(stroke
 				(width 0.12)
@@
 		(fp_line
 			(start -1.62 6)
-			(end -1.62 8.73)
-			(stroke
-				(width 0.12)
-				(type solid)
-			)
-			(layer "F.SilkS")
-		)
-		(fp_line
-			(start -1.62 8.73)
-			(end 7.57 8.73)
+			(end -1.62 8.26)
 			(stroke
 				(width 0.12)
@@
 	(footprint "Capacitor_SMD:C_0402_1005Metric"
 		(layer "F.Cu")
-		(at 54.2 67.5)
+		(at 61.1 69.1)
 		(descr "Capacitor SMD 0402 (1005 Metric), square (rectangular) end terminal, IPC-7351 nominal, (Body size source: IPC-SM-782 page 76, https://www.pcb-3d.com/wordpress/wp-content/uploads/ipc-sm-782a_amendment_1_and_2.pdf)")
 		(tags "capacitor")
@@
 		(duplicate_pad_numbers_are_jumpers no)
 		(fp_line
+			(start 10.03 -1.83)
+			(end 1.81 -1.83)
+			(stroke
+				(width 0.12)
+				(type default)
+			)
+			(layer "F.SilkS")
+		)
+		(fp_line
+			(start 1.81 -1.83)
+			(end 1.81 4.33)
+			(stroke
+				(width 0.12)
+				(type default)
+			)
+			(layer "F.SilkS")
+		)
+		(fp_line
 			(start 0.3 -1.534264)
 			(end -0.3 -1.534264)
@@
 			(layer "F.SilkS")
 		)
-		(fp_rect
-			(start 1.81 -1.83)
-			(end 10.49 4.33)
+		(fp_line
+			(start 1.81 4.33)
+			(end 10.03 4.33)
 			(stroke
 				(width 0.12)
-				(type solid)
+				(type default)
 			)
-			(fill no)
 			(layer "F.SilkS")
 		)
@@
 		(duplicate_pad_numbers_are_jumpers no)
 		(fp_line
+			(start 10.03 -1.83)
+			(end 1.81 -1.83)
+			(stroke
+				(width 0.12)
+				(type default)
+			)
+			(layer "F.SilkS")
+		)
+		(fp_line
+			(start 1.81 -1.83)
+			(end 1.81 4.33)
+			(stroke
+				(width 0.12)
+				(type default)
+			)
+			(layer "F.SilkS")
+		)
+		(fp_line
 			(start 0.3 -1.534264)
 			(end -0.3 -1.534264)
@@
 			(layer "F.SilkS")
 		)
-		(fp_rect
-			(start 1.81 -1.83)
-			(end 10.49 4.33)
+		(fp_line
+			(start 1.81 4.33)
+			(end 10.03 4.33)
 			(stroke
 				(width 0.12)
-				(type solid)
+				(type default)
 			)
-			(fill no)
 			(layer "F.SilkS")
 		)
@@
 		(duplicate_pad_numbers_are_jumpers no)
 		(fp_line
+			(start 10.03 -1.83)
+			(end 1.81 -1.83)
+			(stroke
+				(width 0.12)
+				(type default)
+			)
+			(layer "F.SilkS")
+		)
+		(fp_line
+			(start 1.81 -1.83)
+			(end 1.81 6.83)
+			(stroke
+				(width 0.12)
+				(type default)
+			)
+			(layer "F.SilkS")
+		)
+		(fp_line
 			(start 0.3 -1.534264)
 			(end -0.3 -1.534264)
@@
 			(layer "F.SilkS")
 		)
-		(fp_rect
-			(start 1.81 -1.83)
-			(end 10.49 6.83)
+		(fp_line
+			(start 1.81 6.83)
+			(end 10.03 6.83)
 			(stroke
 				(width 0.12)
-				(type solid)
+				(type default)
 			)
-			(fill no)
 			(layer "F.SilkS")
 		)
@@
 	)
 	(segment
-		(start 54.68 68)
-		(end 56.3 68.35)
-		(width 0.3)
-		(layer "F.Cu")
-		(net "PGND")
-	)
-	(segment
 		(start 61.4 59.05)
 		(end 62.05 59.05)
@@
 	)
 	(segment
+		(start 61.58 69.1)
+		(end 61.9 69.1)
+		(width 0.3)
+		(layer "F.Cu")
+		(net "PGND")
+	)
+	(segment
 		(start 60 63.15)
 		(end 60 62.95)
@@
 	)
 	(segment
-		(start 54.68 67.5)
-		(end 54.68 68)
-		(width 0.3)
-		(layer "F.Cu")
-		(net "PGND")
-	)
-	(segment
 		(start 60 64.3)
 		(end 60 63.15)
@@
 	)
 	(via
+		(at 61.9 69.1)
+		(size 0.7)
+		(drill 0.3)
+		(layers "F.Cu" "B.Cu")
+		(net "PGND")
+	)
+	(via
 		(at 72 59.05)
 		(size 0.5)
@@
 	)
 	(segment
-		(start 53.72 67.5)
-		(end 51.6 67.5)
+		(start 60.62 69.1)
+		(end 59.7 69.4)
 		(width 0.2)
 		(layer "F.Cu")
@@
 	)
 	(segment
-		(start 51.6 67.5)
-		(end 51.6 68.5)
-		(width 0.2)
-		(layer "F.Cu")
-		(net "VIN1")
-	)
-	(segment
 		(start 43.6 70.1)
 		(end 43.6 69.4)
@@
 	)
 	(via
-		(at 58.6 69.4)
-		(size 0.5)
-		(drill 0.3)
-		(layers "F.Cu" "B.Cu")
-		(net "VIN1")
-	)
-	(via
-		(at 51.6 68.5)
-		(size 0.5)
-		(drill 0.3)
-		(layers "F.Cu" "B.Cu")
-		(net "VIN1")
-	)
-	(via
 		(at 43.6 70.1)
 		(size 0.7)
@@
 	)
 	(segment
-		(start 51.6 68.5)
-		(end 51.6 74)
+		(start 59.7 69.4)
+		(end 60.5 69.4)
 		(width 0.2)
 		(layer "In2.Cu")
@@
 		(layer "In2.Cu")
 		(net "VIN1")
-	)
-	(segment
-		(start 58.6 69.4)
-		(end 60.5 69.4)
-		(width 0.2)
-		(layer "In2.Cu")
-		(net "VIN1")

Commit message: phase 4.7
Routing:
- net GND: track 0.00 -> 17.8 mm, vias 0 -> 2
- net PGND: track 30.0 -> 35.6 mm, vias 47 -> 49
- net /CHG_GATE: track 0.00 -> 3.45 mm
Changed lines of the file:
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@@
+	)
+	(segment
+		(start 78.7375 62.3)
+		(end 77.8 62.3)
+		(width 0.3)
+		(layer "F.Cu")
+		(net "PGND")
 	)
 	(segment
@@
 	)
 	(segment
+		(start 78.9125 66)
+		(end 79.8 66)
+		(width 0.3)
+		(layer "F.Cu")
+		(net "PGND")
+	)
+	(segment
 		(start 63.7 59.65)
 		(end 62.05 59.05)
@@
 	)
 	(segment
+		(start 79.8 66)
+		(end 79.8 69.8)
+		(width 0.3)
+		(layer "F.Cu")
+		(net "PGND")
+	)
+	(segment
 		(start 61.4 59.05)
 		(end 62.05 59.05)
@@
 	)
 	(via
+		(at 77.8 62.3)
+		(size 0.7)
+		(drill 0.3)
+		(layers "F.Cu" "B.Cu")
+		(net "PGND")
+	)
+	(via
 		(at 61.9 69.1)
 		(size 0.7)
@@
 		(at 57.5 68.9)
 		(size 0.5)
+		(drill 0.3)
+		(layers "F.Cu" "B.Cu")
+		(net "PGND")
+	)
+	(via
+		(at 79.8 69.8)
+		(size 0.7)
 		(drill 0.3)
 		(layers "F.Cu" "B.Cu")
@@
 	)
 	(segment
+		(start 78.7375 64.2)
+		(end 77.0875 64.2)
+		(width 0.2)
+		(layer "F.Cu")
+		(net "/CHG_GATE")
+	)
+	(segment
+		(start 77.0875 64.2)
+		(end 77.0875 66)
+		(width 0.2)
+		(layer "F.Cu")
+		(net "/CHG_GATE")
+	)
+	(segment
 		(start 42.4625 49)
 		(end 42.4625 50.5)
@@
 		(net "Net-(C26-Pad1)")
 	)
+	(segment
+		(start 78.2 73.4125)
+		(end 78.2 73.7)
+		(width 0.2)
+		(layer "F.Cu")
+		(net "GND")
+	)
+	(segment
+		(start 65.412499 71.2)
+		(end 66.099999 71.2)
+		(width 0.2)
+		(layer "F.Cu")
+		(net "GND")
+	)
+	(segment
+		(start 77 73.4125)
+		(end 78.2 73.4125)
+		(width 0.2)
+		(layer "F.Cu")
+		(net "GND")
+	)
+	(segment
+		(start 66.099999 71.2)
+		(end 66.5 70.8)
+		(width 0.2)
+		(layer "F.Cu")
+		(net "GND")
+	)
+	(segment
+		(start 66.5 70.8)
+		(end 67 70.8)
+		(width 0.2)
+		(layer "F.Cu")
+		(net "GND")
+	)
+	(via
+		(at 78.2 73.7)
+		(size 0.5)
+		(drill 0.3)
+		(layers "F.Cu" "B.Cu")
+		(net "GND")
+	)
+	(via
+		(at 66.5 70.8)
+		(size 0.5)
+		(drill 0.3)
+		(layers "F.Cu" "B.Cu")
+		(net "GND")
+	)
+	(segment
+		(start 66.5 70.8)
+		(end 66.5 73.7)
+		(width 0.2)
+		(layer "B.Cu")
+		(net "GND")
+	)
+	(segment
+		(start 66.5 73.7)
+		(end 78.2 73.7)
+		(width 0.2)
+		(layer "B.Cu")
+		(net "GND")
+	)
 	(zone
