File: hardware/v4/ups_v4/ups12v_v4.kicad_pcb (KiCad board)
At the start: 4 copper layers, 96 x 70 mm, 154 parts, among them IC1 BQ25798RQMR, J1 ADAPTER 4.75-21V, J2 VSYS OUTPUT, J3 BATTERY 2S/4S, J4 MCU / BIAS INTERFACE, J6 NTC temp sensor, J7 USB-C PROGRAM / NATIVE USB, J8 5V / GND, Q1 AON7528, Q10 AON7528, Q2 AON7528, Q3 PMV16UN, Q4 BC847 INT DOMAIN ISOLATOR, Q5 BC857 MAIN-GATED CHG SOURCE, Q6 BC847 MAIN_VALID SINK, Q7 BC847 MCU CHG ARM SINK, Q8 PMV16UN MAIN_VALID, Q9 PMV16UN TCA_EN, SW1 BOOT / DOWNLOAD, SW2 RESET, U1 ESP32-C3-MINI-1-N4X, U2 TPD2EUSB30A (PROVISIONAL), U3 TPS62933DRLR NORMAL 3V3, U4 AP7361C-33E-13 USB 3V3 LDO, U5 TPS2116DRL NORMAL PRIORITY, U6 TCA9517DGKR REV.D, U7 TPS62933DRLR, U8 LM74700QDBVRQ1

Commit message: checkpoint
Routing:
- net PROG: track 0.00 -> 14.2 mm, vias 0 -> 2
- net BATP: track 0.00 -> 14.2 mm
- net TS: track 0.00 -> 10.0 mm
- net ILIM_HIZ: track 0.00 -> 2.38 mm
- net PGND: track 35.6 -> 35.9 mm, vias 49 -> 50

Commit message: phase 4.7
Routing:
- net REGN: track 1.89 -> 46.1 mm, vias 0 -> 2
- net CE_BIAS: track 0.00 -> 40.2 mm
- net CE_N: track 0.00 -> 27.8 mm

Commit message: phase 4.8
Routing:
- net TS: track 10.0 -> 64.3 mm, vias 0 -> 2
- net GND: track 17.8 -> 67.4 mm
- net REGN: track 46.1 -> 67.5 mm
Changed lines of the file:
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@@
+	)
+	(segment
+		(start 39.1 75.5)
+		(end 39.0875 75.5)
+		(width 0.2)
+		(layer "F.Cu")
+		(net "REGN")
 	)
 	(segment
@@
 	)
 	(segment
+		(start 48.15 73.3)
+		(end 48.1 73.4)
+		(width 0.2)
+		(layer "F.Cu")
+		(net "REGN")
+	)
+	(segment
 		(start 72.1 69.4)
 		(end 71.9 69.05)
@@
 	)
 	(segment
+		(start 50.2 68.4)
+		(end 50.05 68.45)
+		(width 0.2)
+		(layer "F.Cu")
+		(net "REGN")
+	)
+	(segment
 		(start 71.9 69.05)
 		(end 71.75 68.9)
@@
 	)
 	(segment
+		(start 40.4 74.6)
+		(end 39.1 75.5)
+		(width 0.2)
+		(layer "F.Cu")
+		(net "REGN")
+	)
+	(segment
+		(start 47.8 73.6)
+		(end 40.55 74.55)
+		(width 0.2)
+		(layer "F.Cu")
+		(net "REGN")
+	)
+	(segment
+		(start 49.85 68.65)
+		(end 48.15 73.3)
+		(width 0.2)
+		(layer "F.Cu")
+		(net "REGN")
+	)
+	(segment
 		(start 76.45 62.35)
 		(end 76.5 62.35)
@@
 	)
 	(segment
+		(start 48.1 73.4)
+		(end 47.95 73.55)
+		(width 0.2)
+		(layer "F.Cu")
+		(net "REGN")
+	)
+	(segment
 		(start 71.9 70.1)
 		(end 71 71.4125)
@@
 	)
 	(segment
+		(start 47.95 73.55)
+		(end 47.8 73.6)
+		(width 0.2)
+		(layer "F.Cu")
+		(net "REGN")
+	)
+	(segment
+		(start 56.3 66.45)
+		(end 50.2 68.4)
+		(width 0.2)
+		(layer "F.Cu")
+		(net "REGN")
+	)
+	(segment
 		(start 75.75 66.8)
 		(end 75.8 66.75)
@@
 		(start 76.75 62.2)
 		(end 76.85 62.05)
+		(width 0.2)
+		(layer "F.Cu")
+		(net "REGN")
+	)
+	(segment
+		(start 50.05 68.45)
+		(end 49.85 68.65)
+		(width 0.2)
+		(layer "F.Cu")
+		(net "REGN")
+	)
+	(segment
+		(start 40.55 74.55)
+		(end 40.4 74.6)
 		(width 0.2)
 		(layer "F.Cu")
@@
 	)
 	(segment
+		(start 77 71.5875)
+		(end 82 71.5875)
+		(width 0.15)
+		(layer "F.Cu")
+		(net "TS")
+	)
+	(segment
+		(start 101.5 39.5)
+		(end 101.5 38.5)
+		(width 0.15)
+		(layer "F.Cu")
+		(net "TS")
+	)
+	(segment
 		(start 71 69.6)
 		(end 71 69.5875)
@@
 	)
 	(segment
+		(start 71 69.6)
+		(end 71.3 70.05)
+		(width 0.15)
+		(layer "F.Cu")
+		(net "TS")
+	)
+	(segment
+		(start 82 71.5875)
+		(end 82.5 71.0875)
+		(width 0.15)
+		(layer "F.Cu")
+		(net "TS")
+	)
+	(segment
+		(start 77.85 71.5875)
+		(end 77 71.5875)
+		(width 0.15)
+		(layer "F.Cu")
+		(net "TS")
+	)
+	(segment
 		(start 63.25 69.325)
 		(end 64.1 69.525)
@@
 		(width 0.15)
 		(layer "F.Cu")
+		(net "TS")
+	)
+	(segment
+		(start 82.5 66.5)
+		(end 95 54)
+		(width 0.15)
+		(layer "F.Cu")
+		(net "TS")
+	)
+	(segment
+		(start 82.5 71.0875)
+		(end 82.5 66.5)
+		(width 0.15)
+		(layer "F.Cu")
+		(net "TS")
+	)
+	(segment
+		(start 95 46)
+		(end 101.5 39.5)
+		(width 0.15)
+		(layer "F.Cu")
+		(net "TS")
+	)
+	(segment
+		(start 95 54)
+		(end 95 46)
+		(width 0.15)
+		(layer "F.Cu")
+		(net "TS")
+	)
+	(via
+		(at 71.3 70.05)
+		(size 0.5)
+		(drill 0.3)
+		(layers "F.Cu" "B.Cu")
+		(net "TS")
+	)
+	(via
+		(at 77.85 71.5875)
+		(size 0.5)
+		(drill 0.3)
+		(layers "F.Cu" "B.Cu")
+		(net "TS")
+	)
+	(segment
+		(start 71.3 70.05)
+		(end 77.85 71.5875)
+		(width 0.15)
+		(layer "B.Cu")
 		(net "TS")
 	)
@@
 	)
 	(segment
+		(start 78.2 73.4125)
+		(end 78.2 72.5)
+		(width 0.2)
+		(layer "F.Cu")
+		(net "GND")
+	)
+	(segment
+		(start 83 66.7075)
+		(end 95.5 54.2075)
+		(width 0.2)
+		(layer "F.Cu")
+		(net "GND")
+	)
+	(segment
+		(start 95.5 46.2075)
+		(end 102 39.7075)
+		(width 0.2)
+		(layer "F.Cu")
+		(net "GND")
+	)
+	(segment
 		(start 65.412499 71.2)
 		(end 66.099999 71.2)
@@
 		(width 0.2)
 		(layer "F.Cu")
+		(net "GND")
+	)
+	(segment
+		(start 104 39.7075)
+		(end 104 38.5)
+		(width 0.2)
+		(layer "F.Cu")
+		(net "GND")
+	)
+	(segment
+		(start 95.5 54.2075)
+		(end 95.5 46.2075)
+		(width 0.2)
+		(layer "F.Cu")
+		(net "GND")
+	)
+	(segment
+		(start 83 72.5)
+		(end 83 66.7075)
+		(width 0.2)
+		(layer "F.Cu")
+		(net "GND")
+	)
+	(segment
+		(start 78.2 72.5)
+		(end 83 72.5)
+		(width 0.2)
+		(layer "F.Cu")
+		(net "GND")
+	)
+	(segment
+		(start 102 39.7075)
+		(end 104 39.7075)
+		(width 0.2)
+		(layer "F.Cu")

Commit message: phase 4.8a
Parts:
- moved L2 14.0 mm to (49.6, 85.0), turned to -90 degrees
- moved C45 9.14 mm to (56.4, 85.0)
- moved C33 9.06 mm to (54.0, 85.0)
- moved C37 3.98 mm to (50.9, 79.5), turned to -90 degrees
Routing:
- net MAIN_3V3: track 0.00 -> 25.3 mm, vias 0 -> 2
- net PGND: track 35.9 -> 47.3 mm, vias 50 -> 59
- net SYS: track 75.2 -> 85.3 mm
- net /MAIN_FB: track 0.00 -> 9.28 mm
- net /SW_NORMAL: track 0.00 -> 4.79 mm
- net /NORMAL_SS: track 0.00 -> 4.35 mm
- net /NORMAL_EN: track 0.00 -> 4.21 mm
- net /BST_NORMAL: track 0.00 -> 1.26 mm

Commit message: phase 8b
Routing:
- net SYS: track 85.3 -> 137.8 mm, vias 4 -> 7
- net USB3V3: track 0.00 -> 51.7 mm
- net USB_VBUS: track 0.00 -> 26.5 mm
- net MAIN_3V3: track 25.3 -> 40.6 mm, vias 2 -> 4
- net PGND: track 47.3 -> 59.5 mm, vias 59 -> 75
- net MUX_PR1: track 0.00 -> 7.49 mm, vias 0 -> 2
- net MCU3V3: track 0.00 -> 3.48 mm

Commit message: phase 4.9
Routing:
- net MAIN_3V3: track 40.6 -> 161.6 mm, vias 4 -> 10
- net MCU3V3: track 3.48 -> 111.0 mm, vias 0 -> 16
- net I2C_SDA: track 0.00 -> 98.8 mm, vias 0 -> 2
- net I2C_SCL: track 0.00 -> 70.6 mm, vias 0 -> 2
- net ~INT: track 0.00 -> 67.1 mm, vias 0 -> 2
- net PGND: track 59.5 -> 122.6 mm, vias 75 -> 108
- net MCU_EN: track 0.00 -> 54.1 mm, vias 0 -> 2
- net CHG_REQ: track 0.00 -> 52.7 mm, vias 0 -> 2
- net UART_TX: track 0.00 -> 51.9 mm
- net UART_RX: track 0.00 -> 47.3 mm
- net MCU_BOOT: track 0.00 -> 27.3 mm
- net MCU_CHG_ARM: track 0.00 -> 22.9 mm, vias 0 -> 2
- net MCU_SDA: track 0.00 -> 18.4 mm, vias 0 -> 2
- net MCU_INT: track 0.00 -> 17.5 mm, vias 0 -> 3
- net TCA_EN: track 0.00 -> 14.6 mm
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
Commit message: phase 4.10
Routing:
- net PMID: track 19.5 -> 69.5 mm
- net PGND: track 122.6 -> 143.7 mm, vias 108 -> 122
- net VIN1: track 78.4 -> 89.8 mm
- net USB_CC1: track 0.00 -> 8.39 mm, vias 0 -> 1
- net USB_CC2: track 0.00 -> 8.26 mm, vias 0 -> 1
- net BATTERY: track 65.1 -> 72.4 mm, vias 8 -> 10

Commit message: phase 4.13
Parts:
- moved C28 11.1 mm to (114.1, 78.0)
- moved R48 3.44 mm to (96.0, 91.4)
- moved U2 3.14 mm to (115.0, 81.4)
Connections:
- net Net-(U1-USB_D+_/_GPIO19) renamed /USB_MCU_DP
- net Net-(U1-USB_D-_/_GPIO18) renamed /USB_MCU_DN
Routing:
- net USB_DN: track 0.00 -> 32.3 mm
- net USB_DP: track 0.00 -> 32.3 mm
- net /USB_MCU_DP: track 0.00 -> 21.7 mm, vias 0 -> 2
- net /USB_MCU_DN: track 0.00 -> 21.6 mm, vias 0 -> 2
- net MAIN_3V3: track 161.6 -> 159.0 mm
- net USB_VBUS: track 26.5 -> 24.7 mm
- net PGND: track 143.7 -> 145.6 mm
- net USB3V3: track 51.7 -> 53.1 mm
- net Net-(D1-A): track 12.1 -> 11.4 mm
