File: hardware/v4/ups_v4/ups12v_v4.kicad_pcb (KiCad board)
At the start: 4 copper layers, 96 x 70 mm, 154 parts, among them IC1 BQ25798RQMR, J1 ADAPTER 4.75-21V, J2 VSYS OUTPUT, J3 BATTERY 2S/4S, J4 MCU / BIAS INTERFACE, J6 NTC temp sensor, J7 USB-C PROGRAM / NATIVE USB, J8 5V / GND, Q1 AON7528, Q10 AON7528, Q2 AON7528, Q3 PMV16UN, Q4 BC847 INT DOMAIN ISOLATOR, Q5 BC857 MAIN-GATED CHG SOURCE, Q6 BC847 MAIN_VALID SINK, Q7 BC847 MCU CHG ARM SINK, Q8 PMV16UN MAIN_VALID, Q9 PMV16UN TCA_EN, SW1 BOOT / DOWNLOAD, SW2 RESET, U1 ESP32-C3-MINI-1-N4X, U2 TPD2EUSB30A (PROVISIONAL), U3 TPS62933DRLR NORMAL 3V3, U4 AP7361C-33E-13 USB 3V3 LDO, U5 TPS2116DRL NORMAL PRIORITY, U6 TCA9517DGKR REV.D, U7 TPS62933DRLR, U8 LM74700QDBVRQ1

Commit message: phase 4.16
Parts:
- moved R8 0.62 mm to (40.0, 74.9)
Routing:
- net STAT: track 0.00 -> 43.8 mm
- net ~INT: track 67.1 -> 89.5 mm, vias 2 -> 3
- net I2C_SCL: track 70.6 -> 92.8 mm, vias 2 -> 6
- net VIN1: track 90.2 -> 86.3 mm
- net MAIN_3V3: track 159.0 -> 157.4 mm
- net ACDRV1: track 15.5 -> 14.0 mm
- net PMID: track 69.5 -> 68.6 mm
- net CE_N: track 27.8 -> 28.6 mm, vias 0 -> 2
- net CHG_REQ: track 52.7 -> 51.9 mm
- net CE_BIAS: track 40.2 -> 41.0 mm
- net PROG: track 14.2 -> 14.9 mm
- net TS: track 64.3 -> 64.9 mm
- net BATP: track 14.2 -> 14.8 mm
- net REGN: track 67.5 -> 66.9 mm
- net BATTERY: track 72.4 -> 73.0 mm
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
Commit message: phase 4.17
Parts:
- moved L3 12.6 mm to (105.0, 64.2)
- moved C69 11.6 mm to (99.8, 59.5), turned to -90 degrees
- moved C67 9.06 mm to (117.0, 62.0)
- moved Q10 7.50 mm to (113.0, 56.5)
- moved U8 6.86 mm to (117.1, 58.5), turned to 180 degrees
- moved C65 6.09 mm to (113.0, 63.8), turned to -90 degrees
- moved C66 6.04 mm to (110.0, 60.0)
- moved C64 5.94 mm to (109.5, 63.8), turned to -90 degrees
- moved C63 5.70 mm to (108.5, 58.5)
- moved R62 5.12 mm to (98.0, 55.0)
- moved R63 4.93 mm to (98.0, 51.9)
- moved C62 4.71 mm to (104.3, 59.5), turned to -90 degrees
- moved C60 4.54 mm to (96.5, 59.5), turned to -90 degrees
- moved C68 4.30 mm to (113.0, 52.5), turned to 0 degrees
- moved R61 3.44 mm to (105.5, 57.0), turned to 180 degrees
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Routing:
- net SYS: track 138.5 -> 189.5 mm, vias 7 -> 13
- net /F5_5V_OUT: track 0.00 -> 48.1 mm, vias 0 -> 3
- net /F5_RAW: track 0.00 -> 44.8 mm, vias 0 -> 4
- net PGND: track 145.5 -> 162.4 mm, vias 122 -> 137
- net /F5_EN: track 0.00 -> 8.10 mm
- net /F5_FB: track 0.00 -> 6.10 mm
- net /F5_SS: track 0.00 -> 5.93 mm, vias 0 -> 2
- net /F5_VCAP: track 0.00 -> 5.36 mm
- net /F5_SW: track 0.00 -> 3.88 mm
- net /F5_GATE: track 0.00 -> 2.21 mm
- net /F5_BST: track 0.00 -> 2.09 mm
