File: hardware/v4/evidence/phase4-10-owner-editable-scratch/ups12v_v4.kicad_pcb (KiCad board)
At the start: 4 copper layers, 96 x 70 mm, 154 parts, among them IC1 BQ25798RQMR, J1 ADAPTER 4.75-21V, J2 VSYS OUTPUT, J3 BATTERY 2S/4S, J4 MCU / BIAS INTERFACE, J6 NTC temp sensor, J7 USB-C PROGRAM / NATIVE USB, J8 5V / GND, Q1 AON7528, Q10 AON7528, Q2 AON7528, Q3 PMV16UN, Q4 BC847 INT DOMAIN ISOLATOR, Q5 BC857 MAIN-GATED CHG SOURCE, Q6 BC847 MAIN_VALID SINK, Q7 BC847 MCU CHG ARM SINK, Q8 PMV16UN MAIN_VALID, Q9 PMV16UN TCA_EN, SW1 BOOT / DOWNLOAD, SW2 RESET, U1 ESP32-C3-MINI-1-N4X, U2 TPD2EUSB30A (PROVISIONAL), U3 TPS62933DRLR NORMAL 3V3, U4 AP7361C-33E-13 USB 3V3 LDO, U5 TPS2116DRL NORMAL PRIORITY, U6 TCA9517DGKR REV.D, U7 TPS62933DRLR, U8 LM74700QDBVRQ1

Commit message: review
Parts:
- moved U2 13.3 mm to (110.7, 91.4)
- moved C28 11.1 mm to (114.1, 78.0)
- moved R48 3.44 mm to (96.0, 91.4)
Connections:
- net Net-(U1-USB_D+_/_GPIO19) renamed /USB_MCU_DP
- net Net-(U1-USB_D-_/_GPIO18) renamed /USB_MCU_DN
Routing:
- net USB_DP: track 0.00 -> 32.1 mm
- net USB_DN: track 0.00 -> 32.1 mm
- net /USB_MCU_DN: track 0.00 -> 20.5 mm, vias 0 -> 2
- net /USB_MCU_DP: track 0.00 -> 20.4 mm, vias 0 -> 2
- net MAIN_3V3: track 161.6 -> 159.0 mm
- net USB_VBUS: track 26.5 -> 28.6 mm, vias 0 -> 1
- net USB3V3: track 51.7 -> 53.1 mm
- net Net-(D1-A): track 12.1 -> 11.4 mm
- net PGND: track 143.7 -> 144.3 mm, vias 122 -> 123

Commit message: manual fix
Parts:
- moved U2 10.9 mm to (115.0, 81.4)
Routing:
- net USB_VBUS: track 28.6 -> 24.7 mm, vias 1 -> 0
- net /USB_MCU_DP: track 20.4 -> 22.8 mm
- net /USB_MCU_DN: track 20.5 -> 22.7 mm
- net PGND: track 144.3 -> 145.6 mm, vias 123 -> 122
- net MCU_EN: vias 2 -> 1
- net MCU_BOOT_STRAP2: vias 2 -> 1

Commit message: fix
Routing:
- net /USB_MCU_DP: track 22.8 -> 21.7 mm
- net /USB_MCU_DN: track 22.7 -> 21.6 mm
- net MCU_EN: vias 1 -> 2
- net MCU_BOOT_STRAP2: vias 1 -> 2
Changed lines of the file:
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@@
 	)
 	(via
+		(at 86.74 89.5)
+		(size 0.5)
+		(drill 0.3)
+		(layers "F.Cu" "B.Cu")
+		(net "MCU_EN")
+	)
+	(via
 		(at 77.59 87.3)
 		(size 0.5)
@@
 		(net "MCU_BOOT_STRAP2")
 	)
+	(via
+		(at 84.54 89.5)
+		(size 0.5)
+		(drill 0.3)
+		(layers "F.Cu" "B.Cu")
+		(net "MCU_BOOT_STRAP2")
+	)
 	(segment
 		(start 84.49 86.05)
@@
 	)
 	(segment
-		(start 85.598 91.398)
-		(end 84.409822 90.209822)
+		(start 78.8 91)
+		(end 76.900001 91)
 		(width 0.2)
 		(layer "F.Cu")
@@
 	)
 	(segment
-		(start 78.8 91)
-		(end 76.900001 91)
+		(start 83.115644 90.7)
+		(end 79.1 90.7)
 		(width 0.2)
 		(layer "F.Cu")
@@
 	)
 	(segment
-		(start 83.605822 90.209822)
-		(end 83.115644 90.7)
+		(start 79.1 90.7)
+		(end 78.8 91)
 		(width 0.2)
 		(layer "F.Cu")
@@
 	)
 	(segment
-		(start 84.409822 90.209822)
-		(end 83.605822 90.209822)
+		(start 85.598 91.44)
+		(end 85.598 91.398)
 		(width 0.2)
 		(layer "F.Cu")
@@
 	)
 	(segment
-		(start 76.900001 91)
-		(end 76.700001 91.2)
+		(start 85.598 91.398)
+		(end 84.409822 90.209822)
 		(width 0.2)
 		(layer "F.Cu")
@@
 	)
 	(segment
-		(start 79.1 90.7)
-		(end 78.8 91)
+		(start 95.0468 90.9968)
+		(end 95.49 91.44)
 		(width 0.2)
 		(layer "F.Cu")
@@
 	)
 	(segment
-		(start 95.0468 90.9968)
-		(end 95.49 91.44)
+		(start 92.456 91.4)
+		(end 92.8732 90.9828)
 		(width 0.2)
 		(layer "F.Cu")
@@
 	)
 	(segment
-		(start 85.598 92.2528)
-		(end 85.598 91.398)
+		(start 92.8732 90.9828)
+		(end 95.0468 90.9828)
 		(width 0.2)
 		(layer "F.Cu")
@@
 	)
 	(segment
-		(start 92.456 91.4)
-		(end 92.8732 90.9828)
+		(start 76.900001 91)
+		(end 76.700001 91.2)
 		(width 0.2)
 		(layer "F.Cu")
@@
 	)
 	(segment
-		(start 83.115644 90.7)
-		(end 79.1 90.7)
+		(start 83.605822 90.209822)
+		(end 83.115644 90.7)
 		(width 0.2)
 		(layer "F.Cu")
@@
 	)
 	(segment
-		(start 92.8732 90.9828)
-		(end 95.0468 90.9828)
+		(start 95.0468 90.9828)
+		(end 95.0468 90.9968)
 		(width 0.2)
 		(layer "F.Cu")
@@
 	)
 	(segment
-		(start 76.700001 91.2)
-		(end 76.1 91.2)
+		(start 84.409822 90.209822)
+		(end 83.605822 90.209822)
 		(width 0.2)
 		(layer "F.Cu")
@@
 	)
 	(segment
-		(start 95.0468 90.9828)
-		(end 95.0468 90.9968)
+		(start 76.700001 91.2)
+		(end 76.1 91.2)
 		(width 0.2)
 		(layer "F.Cu")
@@
 	)
 	(via
-		(at 85.598 92.2528)
-		(size 1)
-		(drill 0.5)
+		(at 85.598 91.44)
+		(size 0.5)
+		(drill 0.3)
 		(layers "F.Cu" "B.Cu")
 		(net "/USB_MCU_DP")
 	)
 	(segment
-		(start 91.3212 90.2652)
-		(end 92.456 91.4)
+		(start 87.5856 90.2652)
+		(end 91.3212 90.2652)
 		(width 0.2)
 		(layer "B.Cu")
@@
 	)
 	(segment
-		(start 85.598 92.2528)
+		(start 86.4108 91.44)
 		(end 87.5856 90.2652)
 		(width 0.2)
@@
 	)
 	(segment
-		(start 87.5856 90.2652)
-		(end 91.3212 90.2652)
+		(start 91.3212 90.2652)
+		(end 92.456 91.4)
+		(width 0.2)
+		(layer "B.Cu")
+		(net "/USB_MCU_DP")
+	)
+	(segment
+		(start 85.598 91.44)
+		(end 86.4108 91.44)
 		(width 0.2)
 		(layer "B.Cu")
@@
 	(via
 		(at 82.804 89.8652)
-		(size 1)
-		(drill 0.5)
+		(size 0.5)
+		(drill 0.3)
 		(layers "F.Cu" "B.Cu")
 		(net "/USB_MCU_DN")
@@
 	)
 	(segment
-		(start 87.409614 89.8652)
-		(end 82.810499 89.8652)
+		(start 87.104136 90.3224)
+		(end 87.461336 89.9652)
 		(width 0.2)
 		(layer "B.Cu")
@@
 	)
 	(segment
-		(start 89.569614 89.6252)
-		(end 89.569614 89.160035)
+		(start 91.445464 89.9652)
+		(end 91.680264 90.2)
 		(width 0.2)
 		(layer "B.Cu")
@@
 	)
 	(segment
-		(start 87.769614 89.360042)
-		(end 87.769614 89.6252)
+		(start 88.890974 89.9652)
+		(end 89.010974 89.9652)
 		(width 0.2)
 		(layer "B.Cu")
@@
 	)
 	(segment
-		(start 92.456 90.2)
-		(end 91.821686 90.2)
+		(start 91.052041 89.9652)
+		(end 91.445464 89.9652)
 		(width 0.2)
 		(layer "B.Cu")
@@
 	)
 	(segment
-		(start 82.810499 89.8652)
-		(end 82.804 89.8652)
+		(start 89.010974 89.9652)
+		(end 91.052041 89.9652)
 		(width 0.2)
 		(layer "B.Cu")
@@
 	)
 	(segment
-		(start 88.369614 89.6252)
-		(end 88.369614 89.360042)
+		(start 88.290974 89.208835)
+		(end 88.410974 89.208835)
 		(width 0.2)
 		(layer "B.Cu")
@@
 	)
 	(segment
-		(start 88.129614 89.120042)
-		(end 88.009614 89.120042)
-		(width 0.2)
-		(layer "B.Cu")
-		(net "/USB_MCU_DN")
-	)
-	(segment
-		(start 88.969614 89.160035)
-		(end 88.969614 89.6252)
+		(start 91.680264 90.2)
+		(end 92.456 90.2)
 		(width 0.2)
 		(layer "B.Cu")
@@
 	)
 	(segment
-		(start 88.729614 89.8652)
-		(end 88.609614 89.8652)
+		(start 87.461336 89.9652)
+		(end 87.810974 89.9652)
 		(width 0.2)
 		(layer "B.Cu")
@@
 	)
 	(segment
-		(start 89.329614 88.920035)
-		(end 89.209614 88.920035)
+		(start 82.804 89.8652)
+		(end 83.2612 90.3224)
 		(width 0.2)
 		(layer "B.Cu")
@@
 	)
 	(segment
-		(start 91.486886 89.8652)
-		(end 89.809614 89.8652)
+		(start 88.650974 89.448835)
+		(end 88.650974 89.7252)
 		(width 0.2)
 		(layer "B.Cu")
@@
 	)
 	(segment
-		(start 87.529614 89.8652)
-		(end 87.409614 89.8652)
+		(start 88.050974 89.7252)
+		(end 88.050974 89.448835)
 		(width 0.2)
 		(layer "B.Cu")
@@
 	)
 	(segment
-		(start 91.821686 90.2)
-		(end 91.486886 89.8652)
-		(width 0.2)
-		(layer "B.Cu")
-		(net "/USB_MCU_DN")
-	)
-	(arc
-		(start 89.209614 88.920035)
-		(mid 89.039908 88.990329)
-		(end 88.969614 89.160035)
-		(width 0.2)
-		(layer "B.Cu")
-		(net "/USB_MCU_DN")
-	)
-	(arc
-		(start 88.369614 89.360042)
-		(mid 88.29932 89.190336)
-		(end 88.129614 89.120042)
-		(width 0.2)
-		(layer "B.Cu")
-		(net "/USB_MCU_DN")
-	)
-	(arc
-		(start 87.769614 89.6252)
-		(mid 87.69932 89.794906)
-		(end 87.529614 89.8652)
-		(width 0.2)
-		(layer "B.Cu")
-		(net "/USB_MCU_DN")
-	)
-	(arc
-		(start 89.569614 89.160035)
-		(mid 89.49932 88.990329)
-		(end 89.329614 88.920035)
+		(start 83.2612 90.3224)
+		(end 87.104136 90.3224)
 		(width 0.2)
 		(layer "B.Cu")
@@
 	)
 	(arc
-		(start 88.009614 89.120042)
-		(mid 87.839908 89.190336)
-		(end 87.769614 89.360042)
+		(start 88.650974 89.7252)
+		(mid 88.721268 89.894906)
+		(end 88.890974 89.9652)
 		(width 0.2)
 		(layer "B.Cu")
@@
 	)
 	(arc
-		(start 88.609614 89.8652)
-		(mid 88.439908 89.794906)
-		(end 88.369614 89.6252)
+		(start 88.050974 89.448835)
+		(mid 88.121268 89.279129)
+		(end 88.290974 89.208835)
 		(width 0.2)
 		(layer "B.Cu")
@@
 	)
 	(arc
-		(start 88.969614 89.6252)
-		(mid 88.89932 89.794906)
-		(end 88.729614 89.8652)
+		(start 87.810974 89.9652)
+		(mid 87.98068 89.894906)
+		(end 88.050974 89.7252)
 		(width 0.2)
 		(layer "B.Cu")
@@
 	)
 	(arc
-		(start 89.809614 89.8652)
-		(mid 89.639908 89.794906)
-		(end 89.569614 89.6252)
+		(start 88.410974 89.208835)
+		(mid 88.58068 89.279129)
+		(end 88.650974 89.448835)
 		(width 0.2)
 		(layer "B.Cu")
@@
 		(base_line
 			(pts
-				(xy 89.809614 89.8652) (xy 82.810499 89.8652)
+				(xy 87.810974 89.9652) (xy 91.052041 89.9652)
 			)
 		)
 		(base_line_coupled
 			(pts
-				(xy 89.809614 90.2652) (xy 89.942677 90.2652)
+				(xy 87.810974 90.2652) (xy 87.824992 90.2652)
 			)
 		)
 		(corner_radius_percent 80)
 		(end
-			(xy 82.810499 89.8652)
+			(xy 91.052041 89.9652)
 		)
 		(initial_side "left")
@@
 		(last_status "tuned")
 		(last_track_width 0.2)
-		(last_tuning_length 8e-06)
+		(last_tuning_length 1.7e-05)
 		(max_amplitude 1)
 		(min_amplitude 0.2)
 		(min_spacing 0.6)
 		(origin
-			(xy 89.809614 89.8652)
+			(xy 87.810974 89.9652)
 		)
 		(override_custom_rules no)
@@
 		(target_skew_min -0.1)
 		(tuning_mode "diff_pair_skew")
-		(members "076ac8bc-c659-4f53-9948-b66a2e74e165" "0fba4c4d-f5b8-460d-9d88-224ac2ee911b"
-			"2dd1c06f-4754-4389-8e18-3397cdc195f8" "30789723-8b54-470c-8f53-bf236629846a"
-			"541bc853-5f13-4926-938d-c5d3e3279abc" "7981895e-656c-4d6f-8528-53936672ec26"
-			"7b0e6876-4d53-442c-83c7-0c4497314e4a" "82562151-6420-4c3d-8967-bea1530006c7"
-			"86a4af19-c959-4628-a4bb-969f062ee74a" "8d0ef3f4-9122-4d33-b505-1d16c39b7d5a"
-			"98c79f31-aec0-48c3-b5a0-f4545dc14b66" "a360c0c7-b0dc-417a-a137-d63b23d7c6b4"
-			"babff2c3-34b6-4991-a8ba-f152c0a7848c" "e6c4b52b-4020-4cb4-838e-817f15843ac2"
-			"e9b260ff-edae-4ef6-92fe-e75debcd293c" "f89c6aaf-5879-4961-8ddd-afe4eb0ba733"
-			"fbf71d93-d5c3-4c95-813c-96551e126ea1"
+		(members "180d1150-5e2c-4de1-be9b-57427eb4b8a8" "20ef91d4-8320-400e-969d-c3e5225248f6"
+			"224746b0-6553-4d5e-9172-2cc597d5d0af" "2de728ef-cb8f-43a8-b2ce-7a7810899460"
+			"50ec0e66-4f18-4b4a-882e-51e8d8370a18" "66f6b7d1-2589-4f1a-bce6-14a1b658a339"
+			"cd8a830c-7b0f-40f1-85b0-015598b0fc35" "d74d032c-5da6-4e24-95b6-e9c7e303bccc"
+			"daccc51d-9405-4b25-977f-dac8357f75d3"
 		)
 	)
