File: hardware/v4/evidence/phase4-14-owner-walkaround/ups12v_v4.kicad_pcb (KiCad board)
At the start: 4 copper layers, 96 x 70 mm, 154 parts, among them IC1 BQ25798RQMR, J1 ADAPTER 4.75-21V, J2 VSYS OUTPUT, J3 BATTERY 2S/4S, J4 MCU / BIAS INTERFACE, J6 NTC temp sensor, J7 USB-C PROGRAM / NATIVE USB, J8 5V / GND, Q1 AON7528, Q10 AON7528, Q2 AON7528, Q3 PMV16UN, Q4 BC847 INT DOMAIN ISOLATOR, Q5 BC857 MAIN-GATED CHG SOURCE, Q6 BC847 MAIN_VALID SINK, Q7 BC847 MCU CHG ARM SINK, Q8 PMV16UN MAIN_VALID, Q9 PMV16UN TCA_EN, SW1 BOOT / DOWNLOAD, SW2 RESET, U1 ESP32-C3-MINI-1-N4X, U2 TPD2EUSB30A (PROVISIONAL), U3 TPS62933DRLR NORMAL 3V3, U4 AP7361C-33E-13 USB 3V3 LDO, U5 TPS2116DRL NORMAL PRIORITY, U6 TCA9517DGKR REV.D, U7 TPS62933DRLR, U8 LM74700QDBVRQ1

Commit message: fix
Routing:
- net BATTERY: track 72.3 -> 73.0 mm
Changed lines of the file:
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@@
+	)
+	(segment
+		(start 63.1 65.5)
+		(end 63.1 64.8)
+		(width 0.6)
+		(layer "In2.Cu")
+		(net "BATTERY")
 	)
 	(segment
